Commit message: [UPDATE]: robotican_description

File: robotican_description/komodo/komodo_base_links/Left_URF_link.xacro (robot description, xacro)
@@ -8,5 +8,5 @@
       <origin rpy="0 0 0" xyz="0 0 0" />
       <geometry>
-        <mesh filename="package://ric_description/komodo/meshes/Left_URF_link.STL" />
+        <mesh filename="package://robotican_description/komodo/meshes/Left_URF_link.STL" />
       </geometry>
       <material name="">
@@ -17,5 +17,5 @@
       <origin rpy="0 0 0" xyz="0 0 0" />
       <geometry>
-        <mesh filename="package://ric_description/komodo/meshes/Left_URF_link.STL" />
+        <mesh filename="package://robotican_description/komodo/meshes/Left_URF_link.STL" />
       </geometry>
     </collision>

File: robotican_description/komodo/komodo_base_links/Right_URF_link.xacro (robot description, xacro)
@@ -8,5 +8,5 @@
       <origin rpy="0 0 0" xyz="0 0 0" />
       <geometry>
-        <mesh filename="package://ric_description/komodo/meshes/Right_URF_link.STL" />
+        <mesh filename="package://robotican_description/komodo/meshes/Right_URF_link.STL" />
       </geometry>
       <material name="">
@@ -17,5 +17,5 @@
       <origin rpy="0 0 0" xyz="0 0 0" />
       <geometry>
-        <mesh filename="package://ric_description/komodo/meshes/Right_URF_link.STL" />
+        <mesh filename="package://robotican_description/komodo/meshes/Right_URF_link.STL" />
       </geometry>
     </collision>
