Commit message: [UPDATE]: merging links

File: robotican_description/komodo/models/komodo_base.xacro (robot description, xacro)
@@ -3,7 +3,5 @@
 <robot name="komodo">
 	<!-- Load all the links  -->
-	<xacro:include filename="$(find robotican_description)/komodo/komodo_base_links/base_link.xacro" />
-	<xacro:include filename="$(find robotican_description)/komodo/komodo_base_links/FR_Wheel_link.xacro" />
-	<xacro:include filename="$(find robotican_description)/komodo/komodo_base_links/FL_Wheel_link.xacro" />
+	<xacro:include filename="$(find robotican_description)/komodo/komodo_base_links/komodo_rover.xacro" />
 	<xacro:include filename="$(find robotican_description)/komodo/komodo_base_links/Front_Camera_link.xacro" />
 	<xacro:include filename="$(find robotican_description)/komodo/komodo_base_links/Asus_Camera_link.xacro" />
@@ -12,33 +10,7 @@
 	<xacro:include filename="$(find robotican_description)/komodo/komodo_base_links/Rear_URF_link.xacro" />
 	<xacro:include filename="$(find robotican_description)/komodo/komodo_base_links/Right_URF_link.xacro" />
-	<xacro:include filename="$(find robotican_description)/komodo/komodo_base_links/RL_Wheel_link.xacro" />
-	<xacro:include filename="$(find robotican_description)/komodo/komodo_base_links/RR_Wheel_link.xacro" />
 	<xacro:include filename="$(find robotican_description)/komodo/komodo_base_links/sensors_unit_link.xacro" />
 	<!--         END         -->
 	<!-- Load all the joints -->
-	<joint name="FR_Wheel_joint" type="fixed">
-    		<origin xyz="0.173999999999995 -0.2009 0" rpy="2.62229105359916E-15 6.9308460464278E-17 1.5707963267949" />
-    		<parent link="base_link" />
-    		<child link="FR_Wheel_link" />
-    		<axis xyz="1 0 0" />
-  	</joint>
-	<joint name="FL_Wheel_joint" type="fixed">
-    		<origin xyz="0.173999999999995 0.2009 0" rpy="-2.62229105359916E-15 6.93084604642783E-17 -1.5707963267949" />
-    		<parent link="base_link" />
-    		<child link="FL_Wheel_link" />
-    		<axis xyz="-1 0 0" />
-  	</joint>
-	<joint name="RR_Wheel_joint" type="fixed">
-    		<origin xyz="-0.156000000000005 -0.2009 0" rpy="2.62229105359916E-15 -1.59433090848306E-31 1.5707963267949" />
-    		<parent link="base_link" />
-    		<child link="RR_Wheel_link" />
-    		<axis xyz="1 0 0" />
-  	</joint>
-	<joint name="RL_Wheel_joint" type="fixed">
-    		<origin xyz="-0.156000000000005 0.2009 0" rpy="-2.62229105359916E-15 -5.57680208627196E-32 -1.5707963267949" />
-    		<parent link="base_link" />
-    		<child link="RL_Wheel_link" />
-    		<axis xyz="-1 0 0" />
-  	</joint>
 	<joint name="Left_URF_joint" type="fixed">
     		<origin xyz="-0.0223133326154785 0.137250000000005 0.138508176066688" rpy="-2.73331335606168E-15 1.59433090848306E-31 1.5707963267949" />
