Commit message: fix pkg

File: robotican_description/komodo/komodo_links/komodo_rover.xacro (robot description, xacro)
@@ -113,5 +113,5 @@
 	<!--         END         -->
 	<!-- Load all the joints -->
-	<joint name="FR_Wheel_joint" type="fixed">
+	<joint name="FR_Wheel_joint" type="continuous">
     		<origin xyz="0.173999999999995 -0.2009 0" rpy="2.62229105359916E-15 6.9308460464278E-17 1.5707963267949" />
     		<parent link="base_link" />
@@ -119,5 +119,5 @@
     		<axis xyz="1 0 0" />
   	</joint>
-	<joint name="FL_Wheel_joint" type="fixed">
+	<joint name="FL_Wheel_joint" type="continuous">
     		<origin xyz="0.173999999999995 0.2009 0" rpy="-2.62229105359916E-15 6.93084604642783E-17 -1.5707963267949" />
     		<parent link="base_link" />
@@ -125,5 +125,5 @@
     		<axis xyz="-1 0 0" />
   	</joint>
-	<joint name="RR_Wheel_joint" type="fixed">
+	<joint name="RR_Wheel_joint" type="continuous">
     		<origin xyz="-0.156000000000005 -0.2009 0" rpy="2.62229105359916E-15 -1.59433090848306E-31 1.5707963267949" />
     		<parent link="base_link" />
@@ -131,5 +131,5 @@
     		<axis xyz="1 0 0" />
   	</joint>
-	<joint name="RL_Wheel_joint" type="fixed">
+	<joint name="RL_Wheel_joint" type="continuous">
     		<origin xyz="-0.156000000000005 0.2009 0" rpy="-2.62229105359916E-15 -5.57680208627196E-32 -1.5707963267949" />
     		<parent link="base_link" />

File: robotican_description/komodo/models/komodo_with_arm.xacro (robot description, xacro)
@@ -2,8 +2,8 @@
 <robot xmlns:xacro="http://www.ros.org/wiki/xacro" name="komodo_with_arm">
 	<!--    BASE ROBOT     -->
-	<xacro:include filename="$(find robotican_description)/komodo/models/komodo_base.xacro" >
+	<xacro:include filename="$(find robotican_description)/komodo/models/komodo_base.xacro" />
 	<!--        END        -->
 	<!--        ARM        -->
-	<xacro:include filename="$(find robotican_description)/robot_arms/dynamixel_arm/arm.xacro" >
+	<xacro:include filename="$(find robotican_description)/robot_arms/dynamixel_arm/arm.xacro" />
 	<!--        END        -->
 	<!--    LOAD JOINTS    -->
@@ -11,7 +11,7 @@
     		<origin xyz="-0.112249972183238 0 0.167160698455407" rpy="3.54761842723405E-15 -3.56763412295181E-15 -3.35371649289343E-30" />
     		<parent link="base_link" />
-    		<child link="Arm_base_link" />
+ga    		<child link="Arm_base_link" />
     		<axis xyz="0 0 1" />
-  	</joint>
+  	</joint>gazebo
 	<!--        END        -->
 </robot>

File: robotican_simulation/models/komodo.xacro (robot description, xacro)
@@ -224,5 +224,5 @@
 				<wheelSeparation>0.5</wheelSeparation>
 				<wheelDiameter>0.2</wheelDiameter>
-				<robotBaseFrame>dummy_link</robotBaseFrame>
+				<robotBaseFrame>base_link</robotBaseFrame>
 				<odometryTopic>diff_driver/odometry</odometryTopic>
 				<odometryFrame>odom_link</odometryFrame>
