Commit message: update

File: robotican_description/robot_arms/dynamixel_arm/arm.xacro (robot description, xacro)
@@ -214,5 +214,5 @@
     		<child link="base_rotation_link" />
     		<axis xyz="0 0 1" />
-    		<limit lower="-1.57079" upper="1.57079" effort="0" velocity="0" />
+    		<limit lower="-1.57079" upper="1.57079" effort="10" velocity="0" />
 	</joint>
 	<joint name="shoulder_joint" type="revolute">
@@ -221,5 +221,5 @@
     		<child link="shoulder_link" />
     		<axis xyz="0 1 0" />
-    		<limit lower="-1.692969" upper="1.692969" effort="0" velocity="0" />
+    		<limit lower="-1.692969" upper="1.692969" effort="2000" velocity="0" />
   	</joint>
 	<joint name="elbow1_joint" type="revolute">
@@ -228,5 +228,5 @@
     		<child link="elbow1_link" />
     		<axis xyz="-0.999999999998754 0 0" />
-    		<limit lower="-2.4434" upper="2.4434" effort="0" velocity="0" />
+    		<limit lower="-2.4434" upper="2.4434" effort="100" velocity="0" />
   	</joint>
 	<joint name="elbow2_joint" type="revolute">
@@ -235,5 +235,5 @@
     		<child link="elbow2_link" />
     		<axis xyz="1 0 0" />
-    		<limit lower="-2.4434" upper="2.4434" effort="0" velocity="0" />
+    		<limit lower="-2.4434" upper="2.4434" effort="10" velocity="0" />
   	</joint>
 	<joint name="wrist_joint" type="revolute">
@@ -242,5 +242,5 @@
     		<child link="wrist_link" />
     		<axis xyz="0 0 0.999999999998754" />
-    		<limit lower="-1.91986" upper="1.91986" effort="0" velocity="0" />
+    		<limit lower="-1.91986" upper="1.91986" effort="10" velocity="0" />
   	</joint>
 	<joint name="left_finger_joint" type="revolute">
@@ -249,5 +249,5 @@
    		<child link="left_finger_link" />
     		<axis xyz="1 0 0" />
-    		<limit lower="-0.87266" upper="0.87266" effort="0" velocity="0" />
+    		<limit lower="-0.87266" upper="0.87266" effort="10" velocity="0" />
   	</joint>
 	<joint name="right_finger_joint" type="revolute">
@@ -256,5 +256,5 @@
     		<child link="right_finger_link" />
     		<axis xyz="1 0 0" />
-    		<limit lower="-0.87266" upper="0.87266" effort="0" velocity="0" />
+    		<limit lower="-0.87266" upper="0.87266" effort="10" velocity="0" />
   	</joint>
 	<joint name="Arm_camera_joint" type="fixed">

File: robotican_simulation/models/komodo.xacro (robot description, xacro)
@@ -4,5 +4,5 @@
 	<xacro:arg name="ns" default="komodo"/>
 	<xacro:arg name="color" default="Grey"/>
-	<xacro:arg name="gazebo" default="false"/>
+	<xacro:arg name="gazebo" default="true"/>
 	<xacro:arg name="arm_camera" default="false"/>
 	<xacro:arg name="front_camera" default="false"/>
@@ -224,5 +224,5 @@
 				<wheelSeparation>0.5</wheelSeparation>
 				<wheelDiameter>0.2</wheelDiameter>
-				<robotBaseFrame>base_link</robotBaseFrame>
+				<robotBaseFrame>dummy_link</robotBaseFrame>
 				<odometryTopic>diff_driver/odometry</odometryTopic>
 				<odometryFrame>odom_link</odometryFrame>
