Commit message: [ADD]: elevator model (ubstable)

File: robotican_description/komodo/komodo_links/komod_elevator_links/komodo_elevator.xacro (robot description, xacro)
@@ -116,10 +116,4 @@
 	<!--         END         -->
 	<!-- Load ALL THE JOINTS -->
-	<joint name="Arm_base_joint" type="fixed">
-		<origin xyz="-0.112249972183238 0 0.167160698455407" rpy="0 0 0" />
-		<parent link="base_link" />
-		<child link="Arm_base_link" />
-		<axis xyz="0 0 0" />
-	</joint>
 	<joint name="elevator_joint" type="prismatic">
 		<origin xyz="0.101457996026178 0 0.0740000000000002" rpy="0 0 0" />

Commit message: [UPDATE]: fix elevator model

File: robotican_description/komodo/komodo_links/komod_elevator_links/komodo_elevator.xacro (robot description, xacro)
@@ -116,4 +116,11 @@
 	<!--         END         -->
 	<!-- Load ALL THE JOINTS -->
+	<joint name="base_rotation_joint" type="revolute">
+		<origin xyz="0.113 0 -0.00400000000000003" rpy="-5.46369598732866E-16 1.34659130519145E-15 -2.1922983760752E-31" />
+		<parent link="elevator_link" />
+		<child link="base_rotation_link" />
+		<axis xyz="0 0 1" />
+		<limit lower="-1.57079" upper="1.57079" effort="10" velocity="0" />
+	</joint>
 	<joint name="elevator_joint" type="prismatic">
 		<origin xyz="0.101457996026178 0 0.0740000000000002" rpy="0 0 0" />

File: robotican_description/komodo/models/komodo_with_arm.xacro (robot description, xacro)
@@ -67,5 +67,5 @@
     		<axis xyz="0 0 1" />
   	</joint>
-  		<joint name="Arm_camera_joint" type="fixed">
+	<joint name="Arm_camera_joint" type="fixed">
     		<origin xyz="-0.0552499999999999 0 0.0340250000000002" rpy="1.60129334747211E-25 2.01127359533543E-16 -1.57079632649567" />
     		<parent link="wrist_link" />

Commit message: update

File: robotican_description/komodo/komodo_links/komod_elevator_links/komodo_elevator.xacro (robot description, xacro)
@@ -117,5 +117,5 @@
 	<!-- Load ALL THE JOINTS -->
 	<joint name="base_rotation_joint" type="revolute">
-		<origin xyz="0.113 0 -0.00400000000000003" rpy="-5.46369598732866E-16 1.34659130519145E-15 -2.1922983760752E-31" />
+		<origin xyz="0.113 0 -0.00400000000000003" rpy="0 0 -3.14" />
 		<parent link="elevator_link" />
 		<child link="base_rotation_link" />
@@ -129,5 +129,5 @@
 		<axis xyz="0 0 1" />
 		<dynamics damping="1000.0" friction="100000.0"/>
-		<limit lower="0" upper="0.50" effort="100" velocity="0.000000000000001" />
+		<limit lower="0" upper="0.50" effort="100" velocity="0.2" />
 	</joint>
 	<joint name="Creative_Camera_joint" type="fixed">

Commit message: [UPDAE]: fix wrist

File: robotican_description/komodo/komodo_links/komod_elevator_links/komodo_elevator.xacro (robot description, xacro)
@@ -132,8 +132,8 @@
 	</joint>
 	<joint name="Creative_Camera_joint" type="fixed">
-		<origin xyz="0.0260250000000002 0 0.0520000000000001" rpy="-1.41059322098675E-37 0 -6.20247191139794E-16" />
+		<origin xyz="0.037 0 0.052" rpy="0.0 -1.57 3.14" />
 		<parent link="wrist_link" />
 		<child link="Creative_Camera_link" />
-		<axis xyz="0 0 0" />
+		<axis xyz="0 0 1" />
 	</joint>
 	<joint name="Rear_Camera_joint" type="fixed">

File: robotican_description/robot_arms/dynamixel_arm/arm.xacro (robot description, xacro)
@@ -211,5 +211,5 @@
   	</joint>
 	<joint name="wrist_joint" type="revolute">
-    		<origin xyz="0 -0.0130999999999997 0.244749999999997" rpy="-4.43972025628984E-16 -3.35842401421639E-15 -1.57079632687657" />
+    		<origin xyz="0 0.0 0.244749999999997" rpy="-4.43972025628984E-16 -3.35842401421639E-15 -1.57079632687657" />
     		<parent link="elbow2_link" />
     		<child link="wrist_link" />
