Commit message: update

File: robotican_description/lizi/lizi_links/lizi_rover.xacro (robot description, xacro)
@@ -113,18 +113,18 @@
 	<!--         END         -->
 	<!-- Load all the joints -->
-	<joint name="FL_Wheel_Joint" type="fixed">
+	<joint name="FL_Wheel_Joint" type="continuous">
     		<origin xyz="0.118 0.1338 0.026" rpy="0 0 -1.3371E-16" />
     		<parent link="base_link" />
     		<child link="FL_Wheel_link" />
-    		<axis xyz="0 -1 0" />
+    		<axis xyz="0 1 0" />
   	</joint>
-	<joint name="RL_Wheel_Joint" type="fixed">
+	<joint name="RL_Wheel_Joint" type="continuous">
     		<origin xyz="-0.118 0.1338 0.026" rpy="0 0 -6.6853E-16" />
     		<parent link="base_link" />
     		<child link="RL_Wheel_link" />
-    		<axis xyz="0 -1 0" />
+    		<axis xyz="0 1 0" />
     		<limit effort="0" velocity="0" />
   	</joint>
-	<joint name="RR_Wheel_Joint" type="fixed">
+	<joint name="RR_Wheel_Joint" type="continuous">
     		<origin xyz="-0.118 -0.1338 0.026" rpy="-1.2938E-16 -1.2938E-15 -6.6853E-16" />
     		<parent link="base_link" />
@@ -132,5 +132,5 @@
     		<axis xyz="0 1 0" />
   	</joint>
-	<joint name="FR_Wheel_Joint" type="fixed">
+	<joint name="FR_Wheel_Joint" type="continuous">
     		<origin xyz="0.118 -0.1338 0.026" rpy="4.4216E-16 -0.0061583 -2.6824E-16" />
     		<parent link="base_link" />

File: robotican_description/lizi/models/lizi_base.xacro (robot description, xacro)
@@ -2,4 +2,5 @@
 <robot xmlns:xacro="http://www.ros.org/wiki/xacro" name="komodo">
 	<!-- Load all the links  -->
+	<xacro:property name="lizi_color" value="0 0.517 0.26 1" />
 	<xacro:include filename="$(find robotican_description)/lizi/lizi_links/lizi_rover.xacro" />
 	<xacro:include filename="$(find robotican_description)/lizi/lizi_links/Asus_Camera_link.xacro" />

Commit message: fix lizi

File: robotican_description/lizi/lizi_links/lizi_rover.xacro (robot description, xacro)
@@ -1,3 +1,3 @@
-<robot name="lizi">
+<robot xmlns:xacro="http://www.ros.org/wiki/ric_gazebo" name="lizi">
 	<!-- Load all the links  -->
 	<link name="base_link">
@@ -113,5 +113,5 @@
 	<!--         END         -->
 	<!-- Load all the joints -->
-	<joint name="FL_Wheel_Joint" type="continuous">
+	<joint name="FL_Wheel_Joint" type="$(arg wheels_type)">
     		<origin xyz="0.118 0.1338 0.026" rpy="0 0 -1.3371E-16" />
     		<parent link="base_link" />
@@ -119,5 +119,5 @@
     		<axis xyz="0 1 0" />
   	</joint>
-	<joint name="RL_Wheel_Joint" type="continuous">
+	<joint name="RL_Wheel_Joint" type="$(arg wheels_type)">
     		<origin xyz="-0.118 0.1338 0.026" rpy="0 0 -6.6853E-16" />
     		<parent link="base_link" />
@@ -126,5 +126,5 @@
     		<limit effort="0" velocity="0" />
   	</joint>
-	<joint name="RR_Wheel_Joint" type="continuous">
+	<joint name="RR_Wheel_Joint" type="$(arg wheels_type)">
     		<origin xyz="-0.118 -0.1338 0.026" rpy="-1.2938E-16 -1.2938E-15 -6.6853E-16" />
     		<parent link="base_link" />
@@ -132,5 +132,5 @@
     		<axis xyz="0 1 0" />
   	</joint>
-	<joint name="FR_Wheel_Joint" type="continuous">
+	<joint name="FR_Wheel_Joint" type="$(arg wheels_type)">
     		<origin xyz="0.118 -0.1338 0.026" rpy="4.4216E-16 -0.0061583 -2.6824E-16" />
     		<parent link="base_link" />

File: robotican_description/lizi/models/lizi_base.xacro (robot description, xacro)
@@ -2,8 +2,12 @@
 <robot xmlns:xacro="http://www.ros.org/wiki/xacro" name="komodo">
 	<!-- Load all the links  -->
+	<xacro:arg name="wheels_type" default="fixed"/>
+	<xacro:arg name="have_pan_tilt" default="false"/>
 	<xacro:property name="lizi_color" value="0 0.517 0.26 1" />
 	<xacro:include filename="$(find robotican_description)/lizi/lizi_links/lizi_rover.xacro" />
-	<xacro:include filename="$(find robotican_description)/lizi/lizi_links/Asus_Camera_link.xacro" />
-	<xacro:include filename="$(find robotican_description)/lizi/lizi_links/Asus_Pan_link.xacro" />
+	<xacro:if value="$(arg have_pan_tilt)">
+		<xacro:include filename="$(find robotican_description)/lizi/lizi_links/Asus_Camera_link.xacro" />
+		<xacro:include filename="$(find robotican_description)/lizi/lizi_links/Asus_Pan_link.xacro" />
+	</xacro:if>
 	<xacro:include filename="$(find robotican_description)/lizi/lizi_links/Camera_link.xacro" />
 	<xacro:include filename="$(find robotican_description)/lizi/lizi_links/Laser_link.xacro" />
@@ -13,18 +17,20 @@
 	<!--         END         -->
 	<!-- Load all the joints -->
-	<joint name="Asus_Pan_Joint" type="fixed">
-    		<origin xyz="0.081249 0 0.092091" rpy="2.1253E-16 8.5011E-16 0" />
-    		<parent link="base_link" />
-    		<child link="Asus_Pan_link" />
-    		<axis xyz="0 0 -1" />
-    		<limit effort="0" velocity="0" />
-  	</joint>
-	<joint name="Asus_Tilt_Joint" type="fixed">
-    		<origin xyz="-0.0004889 -0.00041349 0.08" rpy="0 0 0" />
-    		<parent link="Asus_Pan_link" />
-    		<child link="Asus_Camera_link" />
-    		<axis xyz="0 1 0" />
-    		<limit effort="0" velocity="0" />
-  	</joint>
+	<xacro:if value="$(arg have_pan_tilt)">
+		<joint name="Asus_Pan_Joint" type="fixed">
+	    		<origin xyz="0.081249 0 0.092091" rpy="2.1253E-16 8.5011E-16 0" />
+	    		<parent link="base_link" />
+	    		<child link="Asus_Pan_link" />
+	    		<axis xyz="0 0 -1" />
+	    		<limit effort="0" velocity="0" />
+	  	</joint>
+		<joint name="Asus_Tilt_Joint" type="fixed">
+	    		<origin xyz="-0.0004889 -0.00041349 0.08" rpy="0 0 0" />
+	    		<parent link="Asus_Pan_link" />
+	    		<child link="Asus_Camera_link" />
+	    		<axis xyz="0 1 0" />
+	    		<limit effort="0" velocity="0" />
+	  	</joint>
+	</xacro:if>
 	<joint name="Right_URF_Joint" type="fixed">
     		<origin xyz="-0.0074577 -0.1055 0.07895" rpy="0 2.6072E-16 -1.57" />
