Commit message: update

File: robotican_description/robot_arms/h_arm_urdfV3/robots/h_arm_urdf.URDF (robot description, URDF)
Before this commit: robot h_arm_urdf, 9 links, 8 joints
Links:
- link arm_base_link: geometry collision mesh filename=package://robotican_description/robot_arms/h_arm_urdfV3/mes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; visual mesh filename=package://robotican_description/robot_arms/h_arm_urdfV3/mes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
- link arm_rotation1_link: geometry collision mesh filename=package://robotican_description/robot_arms/h_arm_urdfV3/mes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; visual mesh filename=package://robotican_description/robot_arms/h_arm_urdfV3/mes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
- link arm_rotation2_link: geometry collision mesh filename=package://robotican_description/robot_arms/h_arm_urdfV3/mes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; visual mesh filename=package://robotican_description/robot_arms/h_arm_urdfV3/mes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
- link arm_shoulder1_link: geometry collision mesh filename=package://robotican_description/robot_arms/h_arm_urdfV3/mes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; visual mesh filename=package://robotican_description/robot_arms/h_arm_urdfV3/mes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
- link arm_shoulder2_link: geometry collision mesh filename=package://robotican_description/robot_arms/h_arm_urdfV3/mes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; visual mesh filename=package://robotican_description/robot_arms/h_arm_urdfV3/mes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
- link arm_shoulder3_link: geometry collision mesh filename=package://robotican_description/robot_arms/h_arm_urdfV3/mes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; visual mesh filename=package://robotican_description/robot_arms/h_arm_urdfV3/mes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
- link arm_wrist_link: geometry collision mesh filename=package://robotican_description/robot_arms/h_arm_urdfV3/mes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; visual mesh filename=package://robotican_description/robot_arms/h_arm_urdfV3/mes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
- link gripper_l_link: geometry collision mesh filename=package://robotican_description/robot_arms/h_arm_urdfV3/mes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; visual mesh filename=package://robotican_description/robot_arms/h_arm_urdfV3/mes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
- link gripper_r_link: geometry collision mesh filename=package://robotican_description/robot_arms/h_arm_urdfV3/mes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; visual mesh filename=package://robotican_description/robot_arms/h_arm_urdfV3/mes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

Commit message: update

File: robotican_description/robot_arms/h_arm_urdfV3/robots/h_arm_urdf.URDF (robot description, URDF)
Before this commit: robot h_arm_urdf, 9 links, 8 joints
Joints:
- joint gripper_l_joint: axis 1 0 0 -> -1 0 0; origin xyz=0 -0.021 0.04225 rpy=0 0 0 -> xyz=0 -0.021 0.04225 rpy=0.1 0 0
- joint gripper_r_joint: axis 1 0 0 -> -1 0 0; origin xyz=0 0.021 0.04225 rpy=0 0 0 -> xyz=0 0.021 0.04225 rpy=-0.1 0 0
