Commit message: urdfs

File: robotican_description/armadillo/robots/armadillo.xacro (robot description, xacro)
@@ -1,4 +1,4 @@
 <?xml version="1.0"?>
-<robot xmlns:xacro="http://www.ros.org/wiki/xacro" name="komodo_with_arm">
+<robot xmlns:xacro="http://www.ros.org/wiki/xacro" name="komodo_with_arm" description="Armadillo robot">
 	<!--    BASE ROBOT     -->
 	<xacro:include filename="$(find robotican_description)/armadillo/robots/armadillo_base_urdf.xacro" />

File: robotican_description/armadillo/robots/armadillo_base_urdf.xacro (robot description, xacro)
@@ -1,21 +1,22 @@
+<?xml version="1.0"?>
 <robot
-  name="armadillo_base_urdf">
+  name="armadillo_base_urdf" description="Armadillo robot base">
   <link
     name="base_link">
-       <inertial>
-      <origin
-        xyz="-0.060036 0.00010983 0.15247"
-        rpy="0 0 0" />
-      <mass
-        value="80.721" />
-      <inertia
-        ixx="0.62125"
-        ixy="-9.268E-05"
-        ixz="-0.090032"
-        iyy="0.58453"
-        iyz="5.0258E-05"
-        izz="0.36937" />
-    </inertial>
-    <visual>
+    <inertial>
+      <origin
+        xyz="-0.058417 0.00010778 0.15422"
+        rpy="0 0 0" />
+      <mass
+        value="80.6548" />
+      <inertia
+        ixx="0.61639"
+        ixy="-9.1727E-05"
+        ixz="-0.093044"
+        iyy="0.57997"
+        iyz="5.3231E-05"
+        izz="0.36693" />
+    </inertial>
+   <visual name='chassis'>
       <origin
         xyz="0 0 0"
@@ -31,5 +32,5 @@
       </material>
     </visual>
-    <collision>
+  <!--   <collision name='chassis'>
       <origin
         xyz="0 0 0"
@@ -39,5 +40,31 @@
           filename="package://robotican_description/armadillo/meshes/base_link.STL" />
       </geometry>
-    </collision>
+    </collision> -->
+      <collision name='caster_collision'>
+      <origin
+        xyz="-0.35 0 -0.05"
+        rpy="0 0 0" />
+            <geometry>
+              <sphere radius="0.05"/>
+            </geometry>
+            <surface>
+              <friction>
+                <ode>
+                  <mu>0</mu>
+                  <mu2>0</mu2>
+                  <slip1>1.0</slip1>
+                  <slip2>1.0</slip2>
+                </ode>
+              </friction>
+            </surface>
+          </collision>
+	  <!-- <visual name='caster_visual'>
+	           <origin
+        xyz="-0.35 0 -0.05"
+        rpy="0 0 0" />
+            <geometry>
+	    <sphere radius="0.05"/>
+            </geometry>
+	        </visual>-->
   </link>
   <link

File: robotican_description/armadillo/robots/armadillo_elevator_urdf.xacro (robot description, xacro)
@@ -1,4 +1,5 @@
+<?xml version="1.0"?>
 <robot
-  name="armadillo_elevator_urdf">
+  name="armadillo_elevator_urdf" description="Armadillo robot base">
   <link
     name="base_elevator_link">

File: robotican_description/robot_arms/armadillo_arm_urdf/robots/armadillo_arm_urdf.xacro (robot description, xacro)
@@ -1,4 +1,5 @@
+<?xml version="1.0"?>
 <robot
-  name="armadillo_arm_urdf">
+  name="armadillo_arm_urdf" description="Armadillo robot arm">
   <link
     name="base_arm_link">
@@ -159,17 +160,17 @@
   <link
     name="shoulder2_link">
-    <inertial>
-      <origin
-        xyz="-0.029818 0.0063088 0.1262"
+<inertial>
+      <origin
+        xyz="0.068154 0.0063088 0.11032"
         rpy="0 0 0" />
       <mass
         value="0.47392" />
       <inertia
-        ixx="0.0014121"
-        ixy="2.287E-06"
-        ixz="-9.5386E-06"
+        ixx="0.00093237"
+        ixy="-1.0052E-05"
+        ixz="0.00048929"
         iyy="0.0012859"
-        iyz="-1.6503E-05"
-        izz="0.00043354" />
+        iyz="-1.3286E-05"
+        izz="0.00091329" />
     </inertial>
     <visual>
@@ -217,17 +218,17 @@
   <link
     name="rotation2_link">
-    <inertial>
-      <origin
-        xyz="5.0638E-06 0.003816 0.026357"
+ <inertial>
+      <origin
+        xyz="0.018641 0.003816 0.018634"
         rpy="0 0 0" />
       <mass
         value="0.1635" />
       <inertia
-        ixx="0.00014132"
-        ixy="-3.0872E-09"
-        ixz="1.6669E-08"
+        ixx="0.00012408"
+        ixy="2.4076E-06"
+        ixz="1.7225E-05"
         iyy="8.0775E-05"
-        iyz="3.4079E-06"
-        izz="0.00010687" />
+        iyz="2.4119E-06"
+        izz="0.00012412" />
     </inertial>
     <visual>
@@ -259,5 +260,5 @@
     type="revolute">
     <origin
-      xyz="-0.03 0.006 0.2255"
+      xyz="0.13824 0.006 0.18067"
       rpy="0 0 0" />
     <parent
@@ -275,17 +276,17 @@
   <link
     name="shoulder3_link">
-    <inertial>
-      <origin
-        xyz="3.9349E-11 0.012748 0.069689"
+  <inertial>
+      <origin
+        xyz="0.049277 0.012748 0.049277"
         rpy="0 0 0" />
       <mass
         value="0.15954" />
       <inertia
-        ixx="0.00018198"
-        ixy="2.0995E-13"
-        ixz="-2.3374E-13"
+        ixx="0.00012881"
+        ixy="-3.9839E-06"
+        ixz="5.3169E-05"
         iyy="0.00015335"
-        iyz="-5.6341E-06"
-        izz="7.5641E-05" />
+        iyz="-3.9839E-06"
+        izz="0.00012881" />
     </inertial>
     <visual>
@@ -317,5 +318,5 @@
     type="revolute">
     <origin
-      xyz="0 -0.006 0.0325"
+      xyz="0.022981 -0.006 0.022981"
       rpy="0 0 0" />
     <parent
@@ -335,15 +336,15 @@
     <inertial>
       <origin
-        xyz="-0.00053981 -1.4545E-09 0.035177"
+        xyz="0.024492 -8.9152E-11 0.025256"
         rpy="0 0 0" />
       <mass
         value="0.098822" />
       <inertia
-        ixx="6.6953E-05"
-        ixy="7.8184E-12"
-        ixz="1.6384E-06"
+        ixx="6.2194E-05"
+        ixy="2.1384E-12"
+        ixz="3.1204E-06"
         iyy="3.364E-05"
-        iyz="8.578E-13"
-        izz="6.0712E-05" />
+        iyz="-6.2302E-12"
+        izz="6.5471E-05" />
     </inertial>
     <visual>
@@ -375,5 +376,5 @@
     type="revolute">
     <origin
-      xyz="0 0.012 0.117"
+      xyz="0.082731 0.012 0.082731"
       rpy="0 0 0" />
     <parent
@@ -393,15 +394,15 @@
     <inertial>
       <origin
-        xyz="-8.3267E-17 -0.006351 0.015094"
+        xyz="0.010673 -0.006351 0.010673"
         rpy="0 0 0" />
       <mass
         value="0.017607" />
       <inertia
-        ixx="1.4795E-05"
-        ixy="-6.2017E-21"
-        ixz="-4.0048E-20"
+        ixx="1.0362E-05"
+        ixy="2.1712E-06"
+        ixz="4.4332E-06"
         iyy="1.7314E-05"
-        iyz="3.0706E-06"
-        izz="5.9289E-06" />
+        iyz="2.1712E-06"
+        izz="1.0362E-05" />
     </inertial>
     <visual>
@@ -433,5 +434,5 @@
     type="revolute">
     <origin
-      xyz="0 0.049 0.06425"
+   xyz="0.045432 0.049 0.045432"
       rpy="0 0 0" />
     <parent
@@ -440,5 +441,5 @@
       link="left_finger_link" />
     <axis
-      xyz="1 0 0" />
+           xyz="-0.70711 0 0.70711" />
     <limit
       effort="3.1"
@@ -451,15 +452,15 @@
     <inertial>
       <origin
-        xyz="-6.9389E-17 0.006351 0.015094"
+        xyz="0.010673 0.006351 0.010673"
         rpy="0 0 0" />
       <mass
         value="0.017607" />
       <inertia
-        ixx="1.4795E-05"
-        ixy="1.6233E-20"
-        ixz="-3.4691E-20"
+        ixx="1.0362E-05"
+        ixy="-2.1712E-06"
+        ixz="4.4332E-06"
         iyy="1.7314E-05"
-        iyz="-3.0706E-06"
-        izz="5.9289E-06" />
+        iyz="-2.1712E-06"
+        izz="1.0362E-05" />
     </inertial>
     <visual>
@@ -491,5 +492,5 @@
     type="revolute">
     <origin
-      xyz="0 -0.049 0.06425"
+       xyz="0.045432 -0.049 0.045432"
       rpy="0 0 0" />
     <parent
@@ -498,5 +499,5 @@
       link="right_finger_link" />
     <axis
-      xyz="1 0 0" />
+      xyz="-0.70711 0 0.70711" />
     <limit
       effort="3.1"
@@ -509,5 +510,5 @@
     <inertial>
       <origin
-        xyz="1.4624E-09 0.007331 -0.015404"
+        xyz="1.7297E-09 -0.0057087 -0.016076"
         rpy="0 0 0" />
       <mass
@@ -515,9 +516,9 @@
       <inertia
         ixx="2.6617E-05"
-        ixy="-5.2412E-11"
-        ixz="3.4852E-12"
-        iyy="0.00013363"
-        iyz="-5.4873E-06"
-        izz="0.00012728" />
+        ixy="-3.0698E-11"
+        ixz="3.8544E-11"
+        iyy="0.00013594"
+        iyz="3.1747E-06"
+        izz="0.00012497" />
     </inertial>
     <visual>
@@ -549,5 +550,5 @@
     type="fixed">
     <origin
-      xyz="-0.06355 0 0.041852"
+      xyz="-0.015343 0 0.07453"
       rpy="0 0 -1.5708" />
     <parent

File: robotican_simulation/models/armadillo.xacro (robot description, xacro)
@@ -119,5 +119,5 @@
     </sensor>
 </gazebo>
-	  <!-- hokuyo URG-04LX-UG01-->
+	  <!-- hokuyo URG-04LX-UG01   -->
   <gazebo reference="laser_link">
      <sensor type="ray" name="head_hokuyo_sensor">
@@ -141,8 +141,4 @@
         <noise>
           <type>gaussian</type>
-          <!-- Noise parameters based on published spec for Hokuyo laser
-               achieving "+-30mm" accuracy at range < 10m.  A mean of 0.0m and
-               stddev of 0.01m will put 99.7% of samples within 0.03m of the true
-               reading. -->
           <mean>0.0</mean>
           <stddev>0.01</stddev>
@@ -155,5 +151,5 @@
     </sensor>
   </gazebo>
-  <!-- GPS -->
+  <!-- GPS   -->
    <gazebo>
     <plugin name="GazeboRosGps" filename="libhector_gazebo_ros_gps.so">
@@ -168,5 +164,5 @@
     </plugin>
    </gazebo>
-  <!-- IMU -->
+  <!-- IMU   -->
     <gazebo>
       <plugin name="GazeboRosImu" filename="libhector_gazebo_ros_imu.so">
@@ -179,9 +175,8 @@
       <xyzOffsets>0 0 0</xyzOffsets>
       <rpyOffsets>0 0 0</rpyOffsets>
-      <!-- <interface:position name="imu_position"/> -->
       <material>Gazebo/Red</material>
        </plugin>
   </gazebo>
-  <!-- Magnetic -->
+  <!-- Magnetic   -->
     <gazebo>
       <plugin name="GazeboRosMagnetic" filename="libhector_gazebo_ros_magnetic.so">
@@ -195,5 +190,5 @@
     </plugin>
    </gazebo>
-  <!-- camera -->
+  <!-- cameras  -->
   <gazebo reference="front_cam_link">
     <sensor type="camera" name="front_camera">
@@ -212,7 +207,4 @@
         <noise>
           <type>gaussian</type>
-          <!-- Noise is sampled independently per pixel on each frame.
-               That pixel's noise value is added to each of its color
-               channels, which at that point lie in the range [0,1]. -->
           <mean>0.0</mean>
           <stddev>0.007</stddev>
@@ -235,5 +227,5 @@
     </sensor>
   </gazebo>
-  <!-- wheels -->
+  <!-- joints -->
 	<transmission name="left_wheel_joint_trans">
 		<type>transmission_interface/SimpleTransmission</type>
@@ -353,9 +345,4 @@
 			</actuator>
 	</transmission>
-	<gazebo reference="base_link">
-	<selfCollide>true</selfCollide>
-    <mu1>0.0</mu1>
-    <mu2>0.0</mu2>
-  </gazebo>
 	<gazebo reference="base_elevator_link">
 		<turnGravityOff>true</turnGravityOff>
