Commit message: plugins args

File: robotican_description/robot_arms/armadillo_arm_urdf/robots/armadillo_arm_urdf.xacro (robot description, xacro)
@@ -394,15 +394,15 @@
     <inertial>
       <origin
-        xyz="0.010673 -0.006351 0.010673"
-        rpy="0 0 0" />
-      <mass
-        value="0.017607" />
-      <inertia
-        ixx="1.0362E-05"
-        ixy="2.1712E-06"
-        ixz="4.4332E-06"
-        iyy="1.7314E-05"
-        iyz="2.1712E-06"
-        izz="1.0362E-05" />
+        xyz="0.00970400055113302 -0.00893464825232482 0.00970400055113319"
+        rpy="0 0 0" />
+      <mass
+        value="0.0176065040929193" />
+      <inertia
+        ixx="1.00046883612338E-05"
+        ixy="6.24540883843321E-07"
+        ixz="4.79053968386684E-06"
+        iyy="1.80290992370235E-05"
+        iyz="6.24540883843334E-07"
+        izz="1.00046883612338E-05" />
     </inertial>
     <visual>
@@ -434,5 +434,5 @@
     type="revolute">
     <origin
-   xyz="0.045432 0.049 0.045432"
+    xyz="0.048773 0.045707 0.048773"
       rpy="0 0 0" />
     <parent
@@ -452,15 +452,15 @@
     <inertial>
       <origin
-        xyz="0.010673 0.006351 0.010673"
+        xyz="0.009704 0.0089346 0.009704"
         rpy="0 0 0" />
       <mass
         value="0.017607" />
       <inertia
-        ixx="1.0362E-05"
-        ixy="-2.1712E-06"
-        ixz="4.4332E-06"
-        iyy="1.7314E-05"
-        iyz="-2.1712E-06"
-        izz="1.0362E-05" />
+        ixx="1.0005E-05"
+        ixy="-6.2454E-07"
+        ixz="4.7905E-06"
+        iyy="1.8029E-05"
+        iyz="-6.2454E-07"
+        izz="1.0005E-05" />
     </inertial>
     <visual>
@@ -492,5 +492,5 @@
     type="revolute">
     <origin
-       xyz="0.045432 -0.049 0.045432"
+      xyz="0.048773 -0.045707 0.048773"
       rpy="0 0 0" />
     <parent

File: robotican_simulation/models/armadillo.xacro (robot description, xacro)
@@ -1,177 +1,177 @@
 <?xml version="1.0"?>
 <robot xmlns:xacro="http://www.ros.org/wiki/xacro" name="Armadillo" description="Armadillo robot">
-	<xacro:include filename="$(find robotican_description)/armadillo/robots/armadillo.xacro" />
-	<xacro:arg name="front_camera" default="false"/>
-	<xacro:arg name="urf" default="false"/>
-	<xacro:arg name="imu" default="false"/>
-	<xacro:arg name="gps" default="false"/>
-	<xacro:arg name="lidar" default="false"/>
-	<link name="dummy_link">
-	</link>
-	<joint name="dummy_joint" type="fixed">
-		<origin xyz="0.0 0.0 0.0" rpy="0 0 0" />
-		<parent link="dummy_link" />
-		<child link="base_link" />
-		<axis xyz="0 0 0" />
-	</joint>
-	<gazebo>
-		<plugin name="gazebo_ros_control" filename="libgazebo_ros_control.so">
-		</plugin>
-	</gazebo>
-<xacro:property name="M_PI" value="3.1415926535897931" />
-<xacro:property name="URF_FOV" value="${10.0*M_PI/180}" />
-	<!-- Sonars -->
-<xacro:if value="$(arg urf)">
-<gazebo reference="left_urf_link">
-    <sensor type="ray" name="range">
-        <always_on>true</always_on>
-        <update_rate>10</update_rate>
-        <pose>0 0 0 0 0 0</pose>
-        <visualize>false</visualize>
-        <ray>
-            <scan>
-                <horizontal>
-                    <samples>10</samples>
-                    <resolution>1</resolution>
-                    <min_angle>${-URF_FOV/2.0}</min_angle>
-                    <max_angle>${URF_FOV/2.0}</max_angle>
-                </horizontal>
-		<vertical>
-                    <samples>10</samples>
-                    <resolution>1</resolution>
-                    <min_angle>${-URF_FOV/2.0}</min_angle>
-                    <max_angle>${URF_FOV/2.0}</max_angle>
-                </vertical>
-            </scan>
-            <range>
-                <min>0.01</min>
-                <max>5.0</max>
-                <resolution>0.001</resolution>
-            </range>
-        </ray>
-        <plugin name="gazebo_ros_left_urf_controller" filename="libhector_gazebo_ros_sonar.so">
-        <gaussianNoise>0.0001</gaussianNoise>
-        <topicName>URF/left</topicName>
-        <frameId>left_urf_link</frameId>
-        </plugin>
-    </sensor>
-</gazebo>
-<gazebo reference="right_urf_link">
-    <sensor type="ray" name="range">
-        <always_on>true</always_on>
-        <update_rate>10</update_rate>
-        <pose>0 0 0 0 0 0</pose>
-        <visualize>false</visualize>
-        <ray>
-            <scan>
-                <horizontal>
-                    <samples>10</samples>
-                    <resolution>1</resolution>
-                    <min_angle>${-URF_FOV/2.0}</min_angle>
-                    <max_angle>${URF_FOV/2.0}</max_angle>
-                </horizontal>
-		<vertical>
-                    <samples>10</samples>
-                    <resolution>1</resolution>
-                    <min_angle>${-URF_FOV/2.0}</min_angle>
-                    <max_angle>${URF_FOV/2.0}</max_angle>
-                </vertical>
-            </scan>
-            <range>
-                <min>0.01</min>
-                <max>5.0</max>
-                <resolution>0.01</resolution>
-            </range>
-        </ray>
-        <plugin name="gazebo_ros_left_urf_controller" filename="libhector_gazebo_ros_sonar.so">
-        <gaussianNoise>0.001</gaussianNoise>
-        <topicName>URF/right</topicName>
-        <frameId>right_urf_link</frameId>
-        </plugin>
-    </sensor>
-</gazebo>
-<gazebo reference="rear_urf_link">
-    <sensor type="ray" name="range">
-        <always_on>true</always_on>
-        <update_rate>10</update_rate>
-        <pose>0 0 0 0 0 0</pose>
-        <visualize>false</visualize>
-        <ray>
-            <scan>
-                <horizontal>
-                    <samples>10</samples>
-                    <resolution>1</resolution>
-                    <min_angle>${-URF_FOV/2.0}</min_angle>
-                    <max_angle>${URF_FOV/2.0}</max_angle>
-                </horizontal>
-		<vertical>
-                    <samples>10</samples>
-                    <resolution>1</resolution>
-                    <min_angle>${-URF_FOV/2.0}</min_angle>
-                    <max_angle>${URF_FOV/2.0}</max_angle>
-                </vertical>
-            </scan>
-            <range>
-                <min>0.01</min>
-                <max>5.0</max>
-                <resolution>0.01</resolution>
-            </range>
-        </ray>
-        <plugin name="gazebo_ros_left_urf_controller" filename="libhector_gazebo_ros_sonar.so">
-        <gaussianNoise>0.0001</gaussianNoise>
-        <topicName>URF/rear</topicName>
-        <frameId>rear_urf_link</frameId>
-        </plugin>
-    </sensor>
-</gazebo>
-</xacro:if>
-	  <!-- hokuyo URG-04LX-UG01   -->
-<xacro:if value="$(arg lidar)">
-  <gazebo reference="laser_link">
-     <sensor type="ray" name="head_hokuyo_sensor">
-      <pose>0 0 0 0 0 0</pose>
-      <visualize>false</visualize>
-      <update_rate>10</update_rate>
-      <ray>
-        <scan>
-          <horizontal>
-            <samples>667</samples>
-            <resolution>1</resolution>
-            <min_angle>-1.81</min_angle>
-            <max_angle>1.81</max_angle>
-          </horizontal>
-        </scan>
-        <range>
-          <min>0.02</min>
-          <max>5.6</max>
-          <resolution>0.01</resolution>
-        </range>
-        <noise>
-          <type>gaussian</type>
-          <mean>0.0</mean>
-          <stddev>0.01</stddev>
-        </noise>
-      </ray>
-      <plugin name="gazebo_ros_head_hokuyo_controller" filename="libgazebo_ros_laser.so">
-        <topicName>scan</topicName>
-        <frameName>laser_link</frameName>
+  <xacro:include filename="$(find robotican_description)/armadillo/robots/armadillo.xacro" />
+  <xacro:arg name="front_camera" default="false"/>
+  <xacro:arg name="urf" default="false"/>
+  <xacro:arg name="imu" default="false"/>
+  <xacro:arg name="gps" default="false"/>
+  <xacro:arg name="lidar" default="false"/>
+  <link name="dummy_link">
+  </link>
+  <joint name="dummy_joint" type="fixed">
+    <origin xyz="0.0 0.0 0.0" rpy="0 0 0" />
+    <parent link="dummy_link" />
+    <child link="base_link" />
+    <axis xyz="0 0 0" />
+  </joint>
+  <gazebo>
+    <plugin name="gazebo_ros_control" filename="libgazebo_ros_control.so">
+    </plugin>
+  </gazebo>
+  <xacro:property name="M_PI" value="3.1415926535897931" />
+  <xacro:property name="URF_FOV" value="${10.0*M_PI/180}" />
+  <!-- Sonars -->
+  <xacro:if value="$(arg urf)">
+    <gazebo reference="left_urf_link">
+      <sensor type="ray" name="range">
+	<always_on>true</always_on>
+	<update_rate>10</update_rate>
+	<pose>0 0 0 0 0 0</pose>
+	<visualize>false</visualize>
+	<ray>
+	  <scan>
+	    <horizontal>
+	      <samples>10</samples>
+	      <resolution>1</resolution>
+	      <min_angle>${-URF_FOV/2.0}</min_angle>
+	      <max_angle>${URF_FOV/2.0}</max_angle>
+	    </horizontal>
+	    <vertical>
+	      <samples>10</samples>
+	      <resolution>1</resolution>
+	      <min_angle>${-URF_FOV/2.0}</min_angle>
+	      <max_angle>${URF_FOV/2.0}</max_angle>
+	    </vertical>
+	  </scan>
+	  <range>
+	    <min>0.01</min>
+	    <max>5.0</max>
+	    <resolution>0.001</resolution>
+	  </range>
+	</ray>
+	<plugin name="gazebo_ros_left_urf_controller" filename="libhector_gazebo_ros_sonar.so">
+	  <gaussianNoise>0.0001</gaussianNoise>
+	  <topicName>URF/left</topicName>
+	  <frameId>left_urf_link</frameId>
+	</plugin>
+      </sensor>
+    </gazebo>
+    <gazebo reference="right_urf_link">
+      <sensor type="ray" name="range">
+	<always_on>true</always_on>
+	<update_rate>10</update_rate>
+	<pose>0 0 0 0 0 0</pose>
+	<visualize>false</visualize>
+	<ray>
+	  <scan>
+	    <horizontal>
+	      <samples>10</samples>
+	      <resolution>1</resolution>
+	      <min_angle>${-URF_FOV/2.0}</min_angle>
+	      <max_angle>${URF_FOV/2.0}</max_angle>
+	    </horizontal>
+	    <vertical>
+	      <samples>10</samples>
+	      <resolution>1</resolution>
+	      <min_angle>${-URF_FOV/2.0}</min_angle>
+	      <max_angle>${URF_FOV/2.0}</max_angle>
+	    </vertical>
+	  </scan>
+	  <range>
+	    <min>0.01</min>
+	    <max>5.0</max>
+	    <resolution>0.01</resolution>
+	  </range>
+	</ray>
+	<plugin name="gazebo_ros_left_urf_controller" filename="libhector_gazebo_ros_sonar.so">
+	  <gaussianNoise>0.001</gaussianNoise>
+	  <topicName>URF/right</topicName>
+	  <frameId>right_urf_link</frameId>
+	</plugin>
+      </sensor>
+    </gazebo>
+    <gazebo reference="rear_urf_link">
+      <sensor type="ray" name="range">
+	<always_on>true</always_on>
+	<update_rate>10</update_rate>
+	<pose>0 0 0 0 0 0</pose>
+	<visualize>false</visualize>
+	<ray>
+	  <scan>
+	    <horizontal>
+	      <samples>10</samples>
+	      <resolution>1</resolution>
+	      <min_angle>${-URF_FOV/2.0}</min_angle>
+	      <max_angle>${URF_FOV/2.0}</max_angle>
+	    </horizontal>
+	    <vertical>
+	      <samples>10</samples>
+	      <resolution>1</resolution>
+	      <min_angle>${-URF_FOV/2.0}</min_angle>
+	      <max_angle>${URF_FOV/2.0}</max_angle>
+	    </vertical>
+	  </scan>
+	  <range>
+	    <min>0.01</min>
+	    <max>5.0</max>
+	    <resolution>0.01</resolution>
+	  </range>
+	</ray>
+	<plugin name="gazebo_ros_left_urf_controller" filename="libhector_gazebo_ros_sonar.so">
+	  <gaussianNoise>0.0001</gaussianNoise>
+	  <topicName>URF/rear</topicName>
+	  <frameId>rear_urf_link</frameId>
+	</plugin>
+      </sensor>
+    </gazebo>
+  </xacro:if>
+  <!-- hokuyo URG-04LX-UG01   -->
+  <xacro:if value="$(arg lidar)">
+    <gazebo reference="laser_link">
+      <sensor type="ray" name="head_hokuyo_sensor">
+	<pose>0 0 0 0 0 0</pose>
+	<visualize>false</visualize>
+	<update_rate>10</update_rate>
+	<ray>
+	  <scan>
+	    <horizontal>
+	      <samples>667</samples>
+	      <resolution>1</resolution>
+	      <min_angle>-1.81</min_angle>
+	      <max_angle>1.81</max_angle>
+	    </horizontal>
+	  </scan>
+	  <range>
+	    <min>0.02</min>
+	    <max>5.6</max>
+	    <resolution>0.01</resolution>
+	  </range>
+	  <noise>
+	    <type>gaussian</type>
+	    <mean>0.0</mean>
+	    <stddev>0.01</stddev>
+	  </noise>
+	</ray>
+	<plugin name="gazebo_ros_head_hokuyo_controller" filename="libgazebo_ros_laser.so">
+	  <topicName>scan</topicName>
+	  <frameName>laser_link</frameName>
+	</plugin>
+      </sensor>
+    </gazebo>
+  </xacro:if>
+  <!-- GPS   -->
+  <xacro:if value="$(arg gps)">
+    <gazebo>
+      <plugin name="GazeboRosGps" filename="libhector_gazebo_ros_gps.so">
+	<updateRate>50.0</updateRate>
+	<bodyName>base_link</bodyName>
+	<frameId>base_link</frameId>
+	<topicName>GPS/fix</topicName>
+	<serviceName>SERVICE_GPS</serviceName>
+	<velocityTopicName>GPS/fix_velocity</velocityTopicName>
+	<gaussianNoise>2.89e-08 2.89e-08 2.89e-08</gaussianNoise>
+	<velocityGaussianNoise>2.89e-08 2.89e-08 2.89e-08</velocityGaussianNoise>
       </plugin>
-    </sensor>
-  </gazebo>
-</xacro:if>
-  <!-- GPS   -->
-<xacro:if value="$(arg gps)">
-   <gazebo>
-    <plugin name="GazeboRosGps" filename="libhector_gazebo_ros_gps.so">
-      <updateRate>50.0</updateRate>
-      <bodyName>base_link</bodyName>
-      <frameId>base_link</frameId>
-      <topicName>GPS/fix</topicName>
-      <serviceName>SERVICE_GPS</serviceName>
-      <velocityTopicName>GPS/fix_velocity</velocityTopicName>
-      <gaussianNoise>2.89e-08 2.89e-08 2.89e-08</gaussianNoise>
-      <velocityGaussianNoise>2.89e-08 2.89e-08 2.89e-08</velocityGaussianNoise>
-    </plugin>
-   </gazebo>
+    </gazebo>
   </xacro:if>
   <!-- IMU   -->
@@ -179,187 +179,187 @@
     <gazebo>
       <plugin name="GazeboRosImu" filename="libhector_gazebo_ros_imu.so">
-      <alwaysOn>true</alwaysOn>
-      <updateRate>50.0</updateRate>
-      <bodyName>base_link</bodyName>
-      <frameId>base_link</frameId>
-      <topicName>IMU/data</topicName>
-      <gaussianNoise>2.89e-08</gaussianNoise>
-      <xyzOffsets>0 0 0</xyzOffsets>
-      <rpyOffsets>0 0 0</rpyOffsets>
-      <material>Gazebo/Red</material>
-       </plugin>
-  </gazebo>
-  <!-- Magnetic   -->
+	<alwaysOn>true</alwaysOn>
+	<updateRate>50.0</updateRate>
+	<bodyName>base_link</bodyName>
+	<frameId>base_link</frameId>
+	<topicName>IMU/data</topicName>
+	<gaussianNoise>2.89e-08</gaussianNoise>
+	<xyzOffsets>0 0 0</xyzOffsets>
+	<rpyOffsets>0 0 0</rpyOffsets>
+	<material>Gazebo/Red</material>
+      </plugin>
+    </gazebo>
+    <!-- Magnetic   -->
     <gazebo>
       <plugin name="GazeboRosMagnetic" filename="libhector_gazebo_ros_magnetic.so">
-      <updateRate>50.0</updateRate>
-      <bodyName>base_link</bodyName>
-      <frameId>base_link</frameId>
-      <topicName>IMU/magnetic</topicName>
-      <offset>0 0 0</offset>
-      <drift>0.0 0.0 0.0</drift>
-      <gaussianNoise>1.3e-2 1.3e-2 1.3e-2</gaussianNoise>
-    </plugin>
-   </gazebo>
-</xacro:if>
+	<updateRate>50.0</updateRate>
+	<bodyName>base_link</bodyName>
+	<frameId>base_link</frameId>
+	<topicName>IMU/magnetic</topicName>
+	<offset>0 0 0</offset>
+	<drift>0.0 0.0 0.0</drift>
+	<gaussianNoise>1.3e-2 1.3e-2 1.3e-2</gaussianNoise>
+      </plugin>
+    </gazebo>
+  </xacro:if>
   <!-- cameras  -->
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