Commit message: fixes

File: robotican_armadillo/description/models/armadillo_arm.xacro (robot description, xacro)
@@ -220,15 +220,15 @@
  <inertial>
       <origin
-        xyz="0.018641 0.003816 0.018634"
+        xyz="5.0638E-06 0.003816 0.026357"
         rpy="0 0 0" />
       <mass
         value="0.1635" />
       <inertia
-        ixx="0.00012408"
-        ixy="2.4076E-06"
-        ixz="1.7225E-05"
+        ixx="0.00014132"
+        ixy="-3.0872E-09"
+        ixz="1.6669E-08"
         iyy="8.0775E-05"
-        iyz="2.4119E-06"
-        izz="0.00012412" />
+        iyz="3.4079E-06"
+        izz="0.00010687" />
     </inertial>
     <visual>
@@ -261,5 +261,5 @@
     <origin
       xyz="0.13824 0.006 0.18067"
-      rpy="0 0 0" />
+      rpy="-7.2737E-16 0.7854 -5.1433E-16" />
     <parent
       link="shoulder2_link" />
@@ -276,17 +276,17 @@
   <link
     name="shoulder3_link">
-  <inertial>
-      <origin
-        xyz="0.049277 0.012748 0.049277"
+ <inertial>
+      <origin
+        xyz="3.9874E-11 0.012748 0.069689"
         rpy="0 0 0" />
       <mass
         value="0.15954" />
       <inertia
-        ixx="0.00012881"
-        ixy="-3.9839E-06"
-        ixz="5.3169E-05"
+        ixx="0.00018198"
+        ixy="2.1351E-13"
+        ixz="-2.3815E-13"
         iyy="0.00015335"
-        iyz="-3.9839E-06"
-        izz="0.00012881" />
+        iyz="-5.6341E-06"
+        izz="7.5641E-05" />
     </inertial>
     <visual>
@@ -318,6 +318,6 @@
     type="revolute">
     <origin
-      xyz="0.022981 -0.006 0.022981"
-      rpy="0 0 0" />
+      xyz="0 -0.006 0.0325"
+      rpy="1.3906E-15 0 1.3906E-15" />
     <parent
       link="rotation2_link" />
@@ -336,15 +336,15 @@
     <inertial>
       <origin
-        xyz="0.024492 -8.9152E-11 0.025256"
+        xyz="-0.00053981 -8.915E-11 0.035177"
         rpy="0 0 0" />
       <mass
         value="0.098822" />
       <inertia
-        ixx="6.2194E-05"
-        ixy="2.1384E-12"
-        ixz="3.1204E-06"
+        ixx="6.6953E-05"
+        ixy="5.9175E-12"
+        ixz="1.6384E-06"
         iyy="3.364E-05"
-        iyz="-6.2302E-12"
-        izz="6.5471E-05" />
+        iyz="-2.8933E-12"
+        izz="6.0712E-05" />
     </inertial>
     <visual>
@@ -376,6 +376,6 @@
     type="revolute">
     <origin
-      xyz="0.082731 0.012 0.082731"
-      rpy="0 0 0" />
+      xyz="0 0.012 0.117"
+      rpy="-8.0064E-16 0 -8.0064E-16" />
     <parent
       link="shoulder3_link" />
@@ -394,15 +394,15 @@
     <inertial>
       <origin
-        xyz="0.00970400055113302 -0.00893464825232482 0.00970400055113319"
-        rpy="0 0 0" />
-      <mass
-        value="0.0176065040929193" />
-      <inertia
-        ixx="1.00046883612338E-05"
-        ixy="6.24540883843321E-07"
-        ixz="4.79053968386684E-06"
-        iyy="1.80290992370235E-05"
-        iyz="6.24540883843334E-07"
-        izz="1.00046883612338E-05" />
+        xyz="-5.5511E-17 0.015773 0.034449"
+        rpy="0 0 0" />
+      <mass
+        value="0.017607" />
+      <inertia
+        ixx="1.4795E-05"
+        ixy="-1.1493E-20"
+        ixz="2.9858E-20"
+        iyy="1.8029E-05"
+        iyz="8.8323E-07"
+        izz="5.2141E-06" />
     </inertial>
     <visual>
@@ -434,6 +434,6 @@
     type="revolute">
     <origin
-    xyz="0.048773 0.045707 0.048773"
-      rpy="0 0 0" />
+      xyz="0 0.021 0.04825"
+      rpy="8.0345E-16 -1.1657E-15 8.0345E-16" />
     <parent
       link="wrist_link" />
@@ -441,5 +441,5 @@
       link="left_finger_link" />
     <axis
-           xyz="0.70711 0 -0.70711" />
+      xyz="1 0 0" />
     <limit
       effort="3.1"
@@ -452,15 +452,15 @@
     <inertial>
       <origin
-        xyz="0.009704 0.0089346 0.009704"
+        xyz="2.2204E-16 -0.015773 0.034449"
         rpy="0 0 0" />
       <mass
         value="0.017607" />
       <inertia
-        ixx="1.0005E-05"
-        ixy="-6.2454E-07"
-        ixz="4.7905E-06"
+        ixx="1.4795E-05"
+        ixy="-4.8655E-21"
+        ixz="6.7763E-21"
         iyy="1.8029E-05"
-        iyz="-6.2454E-07"
-        izz="1.0005E-05" />
+        iyz="-8.8323E-07"
+        izz="5.2141E-06" />
     </inertial>
     <visual>
@@ -492,6 +492,6 @@
     type="revolute">
     <origin
-      xyz="0.048773 -0.045707 0.048773"
-      rpy="0 0 0" />
+      xyz="0 -0.021 0.04825"
+      rpy="1.0088E-15 -3.3307E-16 1.0088E-15" />
     <parent
       link="wrist_link" />
@@ -499,5 +499,5 @@
       link="right_finger_link" />
     <axis
-      xyz="0.70711 0 -0.70711" />
+      xyz="1 0 0" />
     <limit
       effort="3.1"
@@ -510,5 +510,5 @@
     <inertial>
       <origin
-        xyz="1.7297E-09 -0.0057087 -0.016076"
+        xyz="1.7297E-09 0.007331 -0.015404"
         rpy="0 0 0" />
       <mass
@@ -516,9 +516,9 @@
       <inertia
         ixx="2.6617E-05"
-        ixy="-3.0698E-11"
-        ixz="3.8544E-11"
-        iyy="0.00013594"
-        iyz="3.1747E-06"
-        izz="0.00012497" />
+        ixy="-4.8961E-11"
+        ixz="5.5477E-12"
+        iyy="0.00013363"
+        iyz="-5.4874E-06"
+        izz="0.00012728" />
     </inertial>
     <visual>
@@ -550,6 +550,6 @@
     type="fixed">
     <origin
-      xyz="-0.015343 0 0.07453"
-      rpy="0 0 -1.5708" />
+      xyz="-0.06355 0 0.041852"
+      rpy="9.4369E-16 7.7003E-16 -1.5708" />
     <parent
       link="wrist_link" />

File: robotican_armadillo/description/models/armadillo_elevator.xacro (robot description, xacro)
@@ -317,3 +317,56 @@
       velocity="5.3" />
   </joint>
+  <link
+    name="kinect2_link">
+    <inertial>
+      <origin
+        xyz="-0.095478 0.0037079 -0.034825"
+        rpy="0 0 0" />
+      <mass
+        value="0.82085" />
+      <inertia
+        ixx="0.00059235"
+        ixy="-1.2194E-06"
+        ixz="2.1546E-05"
+        iyy="0.0041195"
+        iyz="2.6946E-05"
+        izz="0.0039702" />
+    </inertial>
+    <visual>
+      <origin
+        xyz="0 0 0"
+        rpy="0 0 0" />
+      <geometry>
+        <mesh
+          filename="package://robotican_armadillo/description/meshes/Kinect2_link.STL" />
+      </geometry>
+      <material
+        name="">
+        <color
+          rgba="0.79216 0.81961 0.93333 1" />
+      </material>
+    </visual>
+    <collision>
+      <origin
+        xyz="0 0 0"
+        rpy="0 0 0" />
+      <geometry>
+        <mesh
+          filename="package://robotican_armadillo/description/meshes/Kinect2_link.STL" />
+      </geometry>
+    </collision>
+  </link>
+  <joint
+    name="kinect2_joint"
+    type="fixed">
+    <origin
+      xyz="0.0518 -0.095 0.072265"
+      rpy="-1.5708 0 -1.5708" />
+    <parent
+      link="head_tilt_link" />
+    <child
+      link="kinect2_link" />
+    <axis
+      xyz="0 0 0" />
+  </joint>
 </robot>

File: robotican_armadillo/description/models/armadillo_gazebo.xacro (robot description, xacro)
@@ -4,51 +4,57 @@
   <xacro:arg name="front_camera" default="false"/>
   <xacro:arg name="rear_camera" default="false"/>
-  <xacro:arg name="top_depth_camera" default="false"/>
+  <xacro:arg name="kinect2" default="false"/>
   <xacro:arg name="urf" default="false"/>
   <xacro:arg name="imu" default="false"/>
   <xacro:arg name="gps" default="false"/>
   <xacro:arg name="lidar" default="false"/>
-<!--  <link name="dummy_link">
+  <!--  <link name="dummy_link">
   </link>
   <joint name="dummy_joint" type="fixed">
-    <origin xyz="0.0 0.0 0.0" rpy="0 0 0" />
-    <parent link="dummy_link" />
-    <child link="base_link" />
-    <axis xyz="0 0 0" />
+  <origin xyz="0.0 0.0 0.0" rpy="0 0 0" />
+  <parent link="dummy_link" />
+  <child link="base_link" />
+  <axis xyz="0 0 0" />
   </joint>-->
-  <!-- controller manager and hardware interfaces -->
   <!-- kinect 2 -->
-    <xacro:if value="$(arg top_depth_camera)">
-  <gazebo>
-  <plugin name="top_depth_camera_controller" filename="libgazebo_ros_openni_kinect.so">
-    <baseline>0.2</baseline>
-    <alwaysOn>true</alwaysOn>
-    <updateRate>1.0</updateRate>
-    <cameraName>top_depth_camera</cameraName>
-    <imageTopicName>top_depth_camera/depth/image_raw</imageTopicName>
-    <cameraInfoTopicName>top_depth_camera/depth/camera_info</cameraInfoTopicName>
-    <depthImageTopicName>top_depth_camera/depth/image_raw</depthImageTopicName>
-    <depthImageInfoTopicName>top_depth_camera/depth/camera_info</depthImageInfoTopicName>
-    <pointCloudTopicName>top_depth_camera/depth/points</pointCloudTopicName>
-    <frameName>top_depth_camera_link</frameName>
-    <pointCloudCutoff>0.5</pointCloudCutoff>
-    <distortionK1>0.00000001</distortionK1>
-    <distortionK2>0.00000001</distortionK2>
-    <distortionK3>0.00000001</distortionK3>
-    <distortionT1>0.00000001</distortionT1>
-    <distortionT2>0.00000001</distortionT2>
-    <CxPrime>0</CxPrime>
-    <Cx>0</Cx>
-    <Cy>0</Cy>
-    <focalLength>0</focalLength>
-    <hackBaseline>0</hackBaseline>
-  </plugin>
-</gazebo>
- </xacro:if>
-  <gazebo>
-    <plugin name="gazebo_ros_control" filename="libgazebo_ros_control.so">
-		<robotSimType>gazebo_ros_control/RoboticanRobotHWSim</robotSimType>
-    </plugin>
-  </gazebo>
+  <xacro:if value="$(arg kinect2)">
+    <gazebo reference="kinect2_link">
+      <sensor type="depth" name="kinect2">
+	<pose>0 0 0 0 0 0</pose>
+	<visualize>true</visualize>
+	<update_rate>5</update_rate>
+        <camera>
+          <horizontal_fov>${70.0*M_PI/180.0}</horizontal_fov>
+          <image>
+            <format>B8G8R8</format>
+            <width>640</width>
+            <height>480</height>
+          </image>
+          <clip>
+            <near>0.5</near>
+            <far>4.5</far>
+          </clip>
+        </camera>
+	<plugin name="kinect2_controller" filename="libgazebo_ros_openni_kinect.so">
+	  <alwaysOn>true</alwaysOn>
+	  <updateRate>20</updateRate>
+	  <cameraName>kinect2</cameraName>
+	  <imageTopicName>hd/image_color</imageTopicName>
+	  <cameraInfoTopicName>hd/camera_info</cameraInfoTopicName>
+	  <depthImageTopicName>hd/image_depth_rect</depthImageTopicName>
+	  <depthImageCameraInfoTopicName>hd/camera_info</depthImageCameraInfoTopicName>
+	  <pointCloudTopicName>hd/points</pointCloudTopicName>
+	  <frameName>kinect2_link</frameName>
+	  <distortion_k1>0.0</distortion_k1>
+	  <distortion_k2>0.0</distortion_k2>
+	  <distortion_k3>0.0</distortion_k3>
+	  <distortion_t1>0.0</distortion_t1>
+	  <distortion_t2>0.0</distortion_t2>
+	  <pointCloudCutoff>0.4</pointCloudCutoff>
+	  <pointCloudCutoffMax>50.0</pointCloudCutoffMax>
+	</plugin>
+      </sensor>
+    </gazebo>
+  </xacro:if>
   <xacro:property name="M_PI" value="3.1415926535897931" />
   <xacro:property name="URF_FOV" value="${10.0*M_PI/180}" />
@@ -240,5 +246,5 @@
       <sensor type="camera" name="front_camera">
 	<update_rate>30.0</update_rate>
-	<camera name="head">
+	<camera name="front_camera">
 	  <horizontal_fov>1.3962634</horizontal_fov>
 	  <image>
@@ -274,9 +280,9 @@
     </gazebo>
   </xacro:if>
-    <xacro:if value="$(arg rear_camera)">
+  <xacro:if value="$(arg rear_camera)">
     <gazebo reference="rear_cam_link">
       <sensor type="camera" name="rear_camera">
 	<update_rate>30.0</update_rate>
-	<camera name="head">
+	<camera name="rear_camera">
 	  <horizontal_fov>1.3962634</horizontal_fov>
 	  <image>
@@ -312,4 +318,10 @@
     </gazebo>
   </xacro:if>
+      <!-- controller manager and hardware interfaces -->
+  <gazebo>
+    <plugin name="gazebo_ros_control" filename="libgazebo_ros_control.so">
+      <robotSimType>gazebo_ros_control/RoboticanRobotHWSim</robotSimType>
+    </plugin>
+  </gazebo>
   <!-- joints -->
   <transmission name="left_wheel_joint_trans">
@@ -340,8 +352,9 @@
     </actuator>
   </transmission>
+  <!--
   <transmission name="rotation1_joint_trans">
     <type>transmission_interface/SimpleTransmission</type>
     <joint name="rotation1_joint">
-      <hardwareInterface>PosVelJointInterface</hardwareInterface>
+      <hardwareInterface>PositionJointInterface</hardwareInterface>
     </joint>
     <actuator name="rotation1_joint_motor">
@@ -352,5 +365,5 @@
     <type>transmission_interface/SimpleTransmission</type>
     <joint name="shoulder1_joint">
-      <hardwareInterface>PosVelJointInterface</hardwareInterface>
+      <hardwareInterface>PositionJointInterface</hardwareInterface>
     </joint>
     <actuator name="shoulder1_joint_motor">
@@ -361,5 +374,5 @@
     <type>transmission_interface/SimpleTransmission</type>
     <joint name="shoulder2_joint">
-      <hardwareInterface>PosVelJointInterface</hardwareInterface>
+      <hardwareInterface>PositionJointInterface</hardwareInterface>
     </joint>
     <actuator name="shoulder2_joint_motor">
@@ -370,5 +383,5 @@
     <type>transmission_interface/SimpleTransmission</type>
     <joint name="rotation2_joint">
-      <hardwareInterface>PosVelJointInterface</hardwareInterface>
+      <hardwareInterface>PositionJointInterface</hardwareInterface>
     </joint>
     <actuator name="rotation2_joint_motor">
@@ -379,5 +392,5 @@
     <type>transmission_interface/SimpleTransmission</type>
     <joint name="shoulder3_joint">
-      <hardwareInterface>PosVelJointInterface</hardwareInterface>
+      <hardwareInterface>PositionJointInterface</hardwareInterface>
     </joint>
     <actuator name="shoulder3_joint_motor">
@@ -388,9 +401,64 @@
     <type>transmission_interface/SimpleTransmission</type>
     <joint name="wrist_joint">
-      <hardwareInterface>PosVelJointInterface</hardwareInterface>
+      <hardwareInterface>PositionJointInterface</hardwareInterface>
     </joint>
     <actuator name="wrist_joint_motor">
       <mechanicalReduction>1</mechanicalReduction>
     </actuator>
+  </transmission>
+  -->
+  <transmission name="rotation1_joint_trans">
+  <type>transmission_interface/SimpleTransmission</type>
+  <joint name="rotation1_joint">
+  <hardwareInterface>PosVelJointInterface</hardwareInterface>
+  </joint>
+  <actuator name="rotation1_joint_motor">
+  <mechanicalReduction>1</mechanicalReduction>
+  </actuator>
+  </transmission>
+  <transmission name="shoulder1_joint_trans">
+  <type>transmission_interface/SimpleTransmission</type>
+  <joint name="shoulder1_joint">
+  <hardwareInterface>PosVelJointInterface</hardwareInterface>
+  </joint>
+  <actuator name="shoulder1_joint_motor">
+  <mechanicalReduction>1</mechanicalReduction>
+  </actuator>
+  </transmission>
+  <transmission name="shoulder2_joint_trans">
+  <type>transmission_interface/SimpleTransmission</type>
+  <joint name="shoulder2_joint">
+  <hardwareInterface>PosVelJointInterface</hardwareInterface>
+  </joint>
+  <actuator name="shoulder2_joint_motor">
+  <mechanicalReduction>1</mechanicalReduction>
+  </actuator>
+  </transmission>
+  <transmission name="rotation2_joint_trans">
+  <type>transmission_interface/SimpleTransmission</type>
+  <joint name="rotation2_joint">
+  <hardwareInterface>PosVelJointInterface</hardwareInterface>
+  </joint>
+  <actuator name="rotation2_joint_motor">
+  <mechanicalReduction>1</mechanicalReduction>
+  </actuator>
+  </transmission>
+  <transmission name="shoulder3_joint_trans">
+  <type>transmission_interface/SimpleTransmission</type>
+  <joint name="shoulder3_joint">
+  <hardwareInterface>PosVelJointInterface</hardwareInterface>
+  </joint>
+  <actuator name="shoulder3_joint_motor">
+  <mechanicalReduction>1</mechanicalReduction>
+  </actuator>
+  </transmission>
+  <transmission name="wrist_joint_trans">
+  <type>transmission_interface/SimpleTransmission</type>
+  <joint name="wrist_joint">
+  <hardwareInterface>PosVelJointInterface</hardwareInterface>
+  </joint>
+  <actuator name="wrist_joint_motor">
+  <mechanicalReduction>1</mechanicalReduction>
+  </actuator>
   </transmission>
   <transmission name="left_finger_joint_trans">

Commit message: f200

File: robotican_armadillo/description/models/armadillo_arm.xacro (robot description, xacro)
@@ -507,9 +507,9 @@
   </joint>
   <link
-    name="f200_optical_link">
+    name="f200_link">
     <inertial>
       <origin
         xyz="1.7297E-09 0.007331 -0.015404"
-        rpy="0 0 0" />
+        rpy="0 0 -1.5708" />
       <mass
         value="0.092188" />
@@ -525,5 +525,5 @@
       <origin
         xyz="0 0 0"
-        rpy="0 0 0" />
+        rpy="0 0 -1.5708" />
       <geometry>
         <mesh
@@ -539,5 +539,5 @@
       <origin
         xyz="0 0 0"
-        rpy="0 0 0" />
+        rpy="0 0 -1.5708" />
       <geometry>
         <mesh
@@ -547,13 +547,13 @@
   </link>
   <joint
-    name="f200_optical_joint"
+    name="f200_joint"
     type="fixed">
     <origin
       xyz="-0.06355 0 0.041852"
-      rpy="9.4369E-16 7.7003E-16 -1.5708" />
+      rpy="9.4369E-16 7.7003E-16 0" />
     <parent
       link="wrist_link" />
     <child
-      link="f200_optical_link" />
+      link="f200_link" />
     <axis
       xyz="0 0 0" />

File: robotican_armadillo/description/models/armadillo_gazebo.xacro (robot description, xacro)
@@ -11,5 +11,7 @@
   <xacro:arg name="gps" default="false"/>
   <xacro:arg name="lidar" default="false"/>
+    <xacro:arg name="f200" default="false"/>
     <xacro:arg name="kinect2_hz" default="10.0"/>
+      <xacro:arg name="f200_hz" default="10.0"/>
   <!--  <link name="dummy_link">
   </link>
@@ -20,4 +22,51 @@
   <axis xyz="0 0 0" />
   </joint>-->
+    <!-- Optical center of camera -->
+    <link name="f200_optical_center_link" />
+    <joint name="f200_optical_center_joint" type="fixed">
+      <origin xyz="0 0 0" rpy="${-M_PI/2} 0 ${-M_PI/2}" />
+      <parent link="f200_link" />
+      <child link="f200_optical_center_link" />
+    </joint>
+    <gazebo reference="f200_link">
+      <sensor type="depth" name="f200_link">
+        <always_on>true</always_on>
+        <update_rate>$(arg f200_hz)</update_rate>
+        <camera>
+          <horizontal_fov>1.20772254</horizontal_fov>
+          <image>
+            <format>L8</format>
+            <width>640</width>
+            <height>480</height>
+          </image>
+          <clip>
+            <near>0.2</near>
+            <far>1.2</far>
+          </clip>
+        </camera>
+        <plugin name="f200_camera_controller" filename="libgazebo_ros_openni_kinect.so">
+          <alwaysOn>true</alwaysOn>
+          <baseline>0.11</baseline>
+          <updateRate>$(arg f200_hz)</updateRate>
+          <cameraName>f200</cameraName>
+          <imageTopicName>camera/image_raw</imageTopicName>
+          <cameraInfoTopicName>camera/camera_info</cameraInfoTopicName>
+          <depthImageTopicName>depth/disparity</depthImageTopicName>
+          <depthImageCameraInfoTopicName>depth/camera_info</depthImageCameraInfoTopicName>
+          <pointCloudTopicName>depth/points</pointCloudTopicName>
+          <frameName>f200_optical_center_link</frameName>
+          <pointCloudCutoff>0.2</pointCloudCutoff>
+          <pointCloudCutoffMax>1.2</pointCloudCutoffMax>
+          <distortionK1>0.0</distortionK1>
+          <distortionK2>0.0</distortionK2>
+          <distortionK3>0.0</distortionK3>
+          <distortionT1>0.0</distortionT1>
+          <distortionT2>0.0</distortionT2>
+    	  <Cx>320</Cx>
+          <Cy>240</Cy>
+          <focalLength>463.888592</focalLength>
+        </plugin>
+      </sensor>
+    </gazebo>
   <!-- kinect 2 -->
   <xacro:if value="$(arg kinect2)">

Commit message: f200

File: robotican_armadillo/description/models/armadillo_arm.xacro (robot description, xacro)
@@ -510,20 +510,20 @@
     <inertial>
       <origin
-        xyz="1.7297E-09 0.007331 -0.015404"
-        rpy="0 0 -1.5708" />
+        xyz="-0.015404 -1.7297E-09 -0.007331"
+        rpy="${M_PI} 0 0" />
       <mass
         value="0.092188" />
       <inertia
-        ixx="2.6617E-05"
-        ixy="-4.8961E-11"
-        ixz="5.5477E-12"
-        iyy="0.00013363"
-        iyz="-5.4874E-06"
-        izz="0.00012728" />
-    </inertial>
-    <visual>
-      <origin
-        xyz="0 0 0"
-        rpy="0 0 -1.5708" />
+        ixx="0.00012728"
+        ixy="-5.5477E-12"
+        ixz="5.4874E-06"
+        iyy="2.6617E-05"
+        iyz="-4.8961E-11"
+        izz="0.00013363" />
+    </inertial>
+    <visual>
+      <origin
+        xyz="0 0 0"
+        rpy="${M_PI} 0 0" />
       <geometry>
         <mesh
@@ -539,5 +539,5 @@
       <origin
         xyz="0 0 0"
-        rpy="0 0 -1.5708" />
+        rpy="${M_PI} 0 0" />
       <geometry>
         <mesh
@@ -551,5 +551,5 @@
     <origin
       xyz="-0.06355 0 0.041852"
-      rpy="9.4369E-16 7.7003E-16 0" />
+      rpy="0 -1.5708 0" />
     <parent
       link="wrist_link" />
@@ -559,3 +559,27 @@
       xyz="0 0 0" />
   </joint>
+  		<link name="f200_rgb_frame" />
+		<joint name="f200_rgb_joint" type="fixed">
+		  <origin xyz="0 -0.0235 0" rpy="0 0 0" />
+		  <parent link="f200_link" />
+		  <child link="f200_rgb_frame" />
+		</joint>
+		 <link name="f200_rgb_optical_frame" />
+		<joint name="f200_rgb_optical_joint" type="fixed">
+		  <origin xyz="0 0 0" rpy="${-M_PI/2} 0 ${-M_PI/2}" />
+		  <parent link="f200_rgb_frame" />
+		  <child link="f200_rgb_optical_frame" />
+		</joint>
+		<link name="f200_depth_frame" />
+		<joint name="f200_depth_joint" type="fixed">
+		  <origin xyz="0 0.0235 0" rpy="0 0 0" />
+		  <parent link="f200_link" />
+		  <child link="f200_depth_frame" />
+		</joint>
+		<link name="f200_depth_optical_frame" />
+		<joint name="f200_depth_optical_joint" type="fixed">
+		  <origin xyz="0 0 0" rpy="${-M_PI/2} 0 ${-M_PI/2}" />
+		  <parent link="f200_depth_frame" />
+		  <child link="f200_depth_optical_frame" />
+		</joint>
 </robot>

File: robotican_armadillo/description/models/armadillo_gazebo.xacro (robot description, xacro)
@@ -23,12 +23,6 @@
     <!-- Optical center of camera -->
      <xacro:if value="$(arg f200)">
-		<link name="f200_optical_center_link" />
-		<joint name="f200_optical_center_joint" type="fixed">
-		  <origin xyz="0 0 0" rpy="${-M_PI/2} 0 ${-M_PI/2}" />
-		  <parent link="f200_link" />
-		  <child link="f200_optical_center_link" />
-		</joint>
-		<gazebo reference="f200_link">
-		  <sensor type="depth" name="f200_link">
+		<gazebo reference="f200_rgb_frame">
+		  <sensor type="depth" name="f200">
 			<always_on>true</always_on>
 			<update_rate>$(arg f200_hz)</update_rate>
@@ -37,6 +31,6 @@
 			  <image>
 				<format>L8</format>
-				<width>640</width>
-				<height>480</height>
+				<width>1280</width>
+				<height>720</height>
 			  </image>
 			  <clip>
@@ -55,5 +49,5 @@
 			  <depthImageCameraInfoTopicName>depth/camera_info</depthImageCameraInfoTopicName>
 			  <pointCloudTopicName>depth/points</pointCloudTopicName>
-			  <frameName>f200_optical_center_link</frameName>
+			  <frameName>f200_depth_optical_frame</frameName>
 			  <pointCloudCutoff>0.2</pointCloudCutoff>
 			  <pointCloudCutoffMax>1.2</pointCloudCutoffMax>
@@ -63,7 +57,7 @@
 			  <distortionT1>0.0</distortionT1>
 			  <distortionT2>0.0</distortionT2>
-			  <Cx>320</Cx>
+			 <!-- <Cx>320</Cx>
 			  <Cy>240</Cy>
-			  <focalLength>463.888592</focalLength>
+			  <focalLength>463.888592</focalLength> -->
 			</plugin>
 		  </sensor>
