Commit message: f200

File: robotican_armadillo/description/models/armadillo_arm.xacro (robot description, xacro)
@@ -511,5 +511,5 @@
       <origin
         xyz="-0.015404 -1.7297E-09 -0.007331"
-        rpy="${M_PI} 0 0" />
+        rpy="0 0 0" />
       <mass
         value="0.092188" />
@@ -525,5 +525,5 @@
       <origin
         xyz="0 0 0"
-        rpy="${M_PI} 0 0" />
+        rpy="0 0 0" />
       <geometry>
         <mesh
@@ -533,14 +533,13 @@
         name="">
         <color
-          rgba="0.79216 0.81961 0.93333 1" />
-      </material>
-    </visual>
-    <collision>
-      <origin
-        xyz="0 0 0"
-        rpy="${M_PI} 0 0" />
-      <geometry>
-        <mesh
-          filename="package://robotican_armadillo/description/meshes/f200_optical_link.STL" />
+          rgba="0.1 0.1 0.1 1" />
+      </material>
+    </visual>
+    <collision>
+      <origin
+        xyz="0 0 0"
+        rpy="0 0 0" />
+      <geometry>
+        <mesh filename="package://robotican_armadillo/description/meshes/f200_optical_link.STL" />
       </geometry>
     </collision>
@@ -561,5 +560,5 @@
   		<link name="f200_rgb_frame" />
 		<joint name="f200_rgb_joint" type="fixed">
-		  <origin xyz="0 -0.0235 0" rpy="0 0 0" />
+		  <origin xyz="0 0 0" rpy="0 0 0" />
 		  <parent link="f200_link" />
 		  <child link="f200_rgb_frame" />
@@ -573,5 +572,5 @@
 		<link name="f200_depth_frame" />
 		<joint name="f200_depth_joint" type="fixed">
-		  <origin xyz="0 0.0235 0" rpy="0 0 0" />
+		  <origin xyz="0 -0.0235 0" rpy="0 0 0" />
 		  <parent link="f200_link" />
 		  <child link="f200_depth_frame" />

File: robotican_armadillo/description/models/armadillo_base.xacro (robot description, xacro)
@@ -32,19 +32,10 @@
       </material>
     </visual>
-  <!--   <collision name='chassis'>
-      <origin
-        xyz="0 0 0"
-        rpy="0 0 0" />
-      <geometry>
-        <mesh
-          filename="package://robotican_armadillo/description/meshes/base_link.STL" />
-      </geometry>
-    </collision> -->
       <collision name='caster_collision'>
       <origin
-        xyz="-0.35 0 -0.05"
+        xyz="-0.35 0 0"
         rpy="0 0 0" />
             <geometry>
-              <sphere radius="0.05"/>
+              <sphere radius="0.1"/>
             </geometry>
             <surface>
@@ -59,12 +50,12 @@
             </surface>
           </collision>
-	  <!-- <visual name='caster_visual'>
-	           <origin
-        xyz="-0.35 0 -0.05"
+	<!--  <visual name='caster_visual'>
+	 <origin
+        xyz="-0.35 0 0"
         rpy="0 0 0" />
             <geometry>
-	    <sphere radius="0.05"/>
+	    <sphere radius="0.1"/>
             </geometry>
-	        </visual>-->
+	  </visual> -->
   </link>
   <link
@@ -140,22 +131,22 @@
       <origin
         xyz="0 0 0"
-        rpy="0 0 0" />
-      <geometry>
-        <mesh
-          filename="package://robotican_armadillo/description/meshes/left_urf_link.STL" />
-      </geometry>
-      <material
-        name="">
-        <color
-          rgba="0.75294 0.75294 0.75294 1" />
-      </material>
-    </visual>
-    <collision>
-      <origin
-        xyz="0 0 0"
-        rpy="0 0 0" />
-      <geometry>
-        <mesh
-          filename="package://robotican_armadillo/description/meshes/left_urf_link.STL" />
+        rpy="0 ${M_PI/2} 0" />
+      <geometry>
+	<!--  <mesh filename="package://robotican_armadillo/description/meshes/left_urf_link.STL" /> -->
+	<cylinder  length="0.01" radius="0.008"/>
+      </geometry>
+      <material
+        name="">
+        <color
+          rgba="0 0 0 1" />
+      </material>
+    </visual>
+    <collision>
+      <origin
+        xyz="0 0 0"
+        rpy="0 ${M_PI/2} 0" />
+      <geometry>
+       	<!--  <mesh filename="package://robotican_armadillo/description/meshes/left_urf_link.STL" /> -->
+	<cylinder  length="0.01" radius="0.008"/>
       </geometry>
     </collision>
@@ -193,22 +184,22 @@
       <origin
         xyz="0 0 0"
-        rpy="0 0 0" />
-      <geometry>
-        <mesh
-          filename="package://robotican_armadillo/description/meshes/right_urf_link.STL" />
-      </geometry>
-      <material
-        name="">
-        <color
-          rgba="0.75294 0.75294 0.75294 1" />
-      </material>
-    </visual>
-    <collision>
-      <origin
-        xyz="0 0 0"
-        rpy="0 0 0" />
-      <geometry>
-        <mesh
-          filename="package://robotican_armadillo/description/meshes/right_urf_link.STL" />
+        rpy="0 ${M_PI/2} 0" />
+      <geometry>
+  <!--      <mesh filename="package://robotican_armadillo/description/meshes/right_urf_link.STL" /> -->
+	<cylinder  length="0.005" radius="0.008"/>
+      </geometry>
+      <material
+        name="">
+        <color
+          rgba="0 0 0 1" />
+      </material>
+    </visual>
+    <collision>
+      <origin
+        xyz="0 0 0"
+         rpy="0 ${M_PI/2} 0" />
+      <geometry>
+  <!--      <mesh filename="package://robotican_armadillo/description/meshes/right_urf_link.STL" /> -->
+	<cylinder  length="0.005" radius="0.008"/>
       </geometry>
     </collision>
@@ -246,22 +237,22 @@
       <origin
         xyz="0 0 0"
-        rpy="0 0 0" />
-      <geometry>
-        <mesh
-          filename="package://robotican_armadillo/description/meshes/rear_urf_link.STL" />
-      </geometry>
-      <material
-        name="">
-        <color
-          rgba="0.75294 0.75294 0.75294 1" />
-      </material>
-    </visual>
-    <collision>
-      <origin
-        xyz="0 0 0"
-        rpy="0 0 0" />
-      <geometry>
-        <mesh
-          filename="package://robotican_armadillo/description/meshes/rear_urf_link.STL" />
+        rpy="0 ${M_PI/2} 0" />
+      <geometry>
+<!--         <mesh  filename="package://robotican_armadillo/description/meshes/rear_urf_link.STL" /> -->
+	<cylinder  length="0.005" radius="0.008"/>
+      </geometry>
+      <material
+        name="">
+        <color
+          rgba="0 0 0 1" />
+      </material>
+    </visual>
+    <collision>
+      <origin
+        xyz="0 0 0"
+        rpy="0 ${M_PI/2} 0" />
+      <geometry>
+<!--         <mesh filename="package://robotican_armadillo/description/meshes/rear_urf_link.STL" /> -->
+	<cylinder  length="0.01" radius="0.008"/>
       </geometry>
     </collision>

File: robotican_armadillo/description/models/armadillo_gazebo.xacro (robot description, xacro)
@@ -3,4 +3,5 @@
   <xacro:include filename="$(find robotican_armadillo)/description/models/armadillo.xacro" />
   <xacro:property name="URF_FOV" value="${10.0*M_PI/180}" />
+ <xacro:arg name="controllers" default="true"/>
   <xacro:arg name="front_camera" default="false"/>
   <xacro:arg name="rear_camera" default="false"/>
@@ -21,5 +22,4 @@
   <axis xyz="0 0 0" />
   </joint>-->
-    <!-- Optical center of camera -->
      <xacro:if value="$(arg f200)">
 		<gazebo reference="f200_rgb_frame">
@@ -30,7 +30,7 @@
 			  <horizontal_fov>1.20772254</horizontal_fov>
 			  <image>
-				<format>L8</format>
-				<width>1280</width>
-				<height>720</height>
+				<format>R8G8B8</format>
+				<width>640</width>
+				<height>480</height>
 			  </image>
 			  <clip>
@@ -41,10 +41,10 @@
 			<plugin name="f200_camera_controller" filename="libgazebo_ros_openni_kinect.so">
 			  <alwaysOn>true</alwaysOn>
-			  <baseline>0.11</baseline>
+			  <!--  <baseline>0.11</baseline> -->
 			  <updateRate>$(arg f200_hz)</updateRate>
 			  <cameraName>f200</cameraName>
-			  <imageTopicName>camera/image_raw</imageTopicName>
-			  <cameraInfoTopicName>camera/camera_info</cameraInfoTopicName>
-			  <depthImageTopicName>depth/disparity</depthImageTopicName>
+			  <imageTopicName>color/image_raw</imageTopicName>
+			  <cameraInfoTopicName>color/camera_info</cameraInfoTopicName>
+			  <depthImageTopicName>depth/image_raw</depthImageTopicName>
 			  <depthImageCameraInfoTopicName>depth/camera_info</depthImageCameraInfoTopicName>
 			  <pointCloudTopicName>depth/points</pointCloudTopicName>
@@ -167,4 +167,5 @@
 	<xacro:if value="$(arg urf)">
 	  <gazebo reference="left_urf_link">
+	     <material>Gazebo/Black</material>
 	    <sensor type="ray" name="range">
 	      <always_on>true</always_on>
@@ -424,4 +425,5 @@
 	</xacro:if>
 	<!-- controller manager and hardware interfaces -->
+<xacro:if value="$(arg controllers)">
 	<gazebo>
 	  <plugin name="gazebo_ros_control" filename="libgazebo_ros_control.so">
@@ -607,3 +609,22 @@
 	  <turnGravityOff>true</turnGravityOff>
 	</gazebo>
+</xacro:if>
+<gazebo reference="right_urf_link">
+    <material>Gazebo/Black</material>
+  </gazebo>
+  <gazebo reference="left_urf_link">
+    <material>Gazebo/Black</material>
+  </gazebo>
+    <gazebo reference="rear_urf_link">
+    <material>Gazebo/Black</material>
+  </gazebo>
+    <gazebo reference="kinect2_link">
+    <material>Gazebo/Black</material>
+  </gazebo>
+    <gazebo reference="laser_link">
+    <material>Gazebo/Black</material>
+  </gazebo>
+    <gazebo reference="f200_link">
+    <material>Gazebo/Grey</material>
+  </gazebo>
       </robot>
