Commit message: update

File: robotican_armadillo/description/models/armadillo.xacro (robot description, xacro)
@@ -1,4 +1,5 @@
 <?xml version="1.0"?>
-<robot xmlns:xacro="http://www.ros.org/wiki/xacro" name="armadillo_with_arm" description="Armadillo robot">
+	<robot xmlns:xacro="http://www.ros.org/wiki/xacro" name="armadillo_with_arm" description="Armadillo robot">
+	<xacro:property name="M_PI" value="3.1415926535897931" />
 	<!--    BASE ROBOT     -->
 	<xacro:include filename="$(find robotican_armadillo)/description/models/armadillo_base.xacro" />

File: robotican_armadillo/description/models/armadillo_gazebo.xacro (robot description, xacro)
@@ -2,5 +2,4 @@
 <robot xmlns:xacro="http://www.ros.org/wiki/xacro" name="Armadillo" description="Armadillo robot">
   <xacro:include filename="$(find robotican_armadillo)/description/models/armadillo.xacro" />
-  <xacro:property name="M_PI" value="3.1415926535897931" />
   <xacro:property name="URF_FOV" value="${10.0*M_PI/180}" />
   <xacro:arg name="front_camera" default="false"/>
@@ -11,7 +10,7 @@
   <xacro:arg name="gps" default="false"/>
   <xacro:arg name="lidar" default="false"/>
-    <xacro:arg name="f200" default="false"/>
-    <xacro:arg name="kinect2_hz" default="10.0"/>
-      <xacro:arg name="f200_hz" default="10.0"/>
+  <xacro:arg name="f200" default="false"/>
+  <xacro:arg name="kinect2_hz" default="10.0"/>
+  <xacro:arg name="f200_hz" default="10.0"/>
   <!--  <link name="dummy_link">
   </link>
@@ -23,50 +22,52 @@
   </joint>-->
     <!-- Optical center of camera -->
-    <link name="f200_optical_center_link" />
-    <joint name="f200_optical_center_joint" type="fixed">
-      <origin xyz="0 0 0" rpy="${-M_PI/2} 0 ${-M_PI/2}" />
-      <parent link="f200_link" />
-      <child link="f200_optical_center_link" />
-    </joint>
-    <gazebo reference="f200_link">
-      <sensor type="depth" name="f200_link">
-        <always_on>true</always_on>
-        <update_rate>$(arg f200_hz)</update_rate>
-        <camera>
-          <horizontal_fov>1.20772254</horizontal_fov>
-          <image>
-            <format>L8</format>
-            <width>640</width>
-            <height>480</height>
-          </image>
-          <clip>
-            <near>0.2</near>
-            <far>1.2</far>
-          </clip>
-        </camera>
-        <plugin name="f200_camera_controller" filename="libgazebo_ros_openni_kinect.so">
-          <alwaysOn>true</alwaysOn>
-          <baseline>0.11</baseline>
-          <updateRate>$(arg f200_hz)</updateRate>
-          <cameraName>f200</cameraName>
-          <imageTopicName>camera/image_raw</imageTopicName>
-          <cameraInfoTopicName>camera/camera_info</cameraInfoTopicName>
-          <depthImageTopicName>depth/disparity</depthImageTopicName>
-          <depthImageCameraInfoTopicName>depth/camera_info</depthImageCameraInfoTopicName>
-          <pointCloudTopicName>depth/points</pointCloudTopicName>
-          <frameName>f200_optical_center_link</frameName>
-          <pointCloudCutoff>0.2</pointCloudCutoff>
-          <pointCloudCutoffMax>1.2</pointCloudCutoffMax>
-          <distortionK1>0.0</distortionK1>
-          <distortionK2>0.0</distortionK2>
-          <distortionK3>0.0</distortionK3>
-          <distortionT1>0.0</distortionT1>
-          <distortionT2>0.0</distortionT2>
-    	  <Cx>320</Cx>
-          <Cy>240</Cy>
-          <focalLength>463.888592</focalLength>
-        </plugin>
-      </sensor>
-    </gazebo>
+     <xacro:if value="$(arg f200)">
+		<link name="f200_optical_center_link" />
+		<joint name="f200_optical_center_joint" type="fixed">
+		  <origin xyz="0 0 0" rpy="${-M_PI/2} 0 ${-M_PI/2}" />
+		  <parent link="f200_link" />
+		  <child link="f200_optical_center_link" />
+		</joint>
+		<gazebo reference="f200_link">
+		  <sensor type="depth" name="f200_link">
+			<always_on>true</always_on>
+			<update_rate>$(arg f200_hz)</update_rate>
+			<camera>
+			  <horizontal_fov>1.20772254</horizontal_fov>
+			  <image>
+				<format>L8</format>
+				<width>640</width>
+				<height>480</height>
+			  </image>
+			  <clip>
+				<near>0.2</near>
+				<far>1.2</far>
+			  </clip>
+			</camera>
+			<plugin name="f200_camera_controller" filename="libgazebo_ros_openni_kinect.so">
+			  <alwaysOn>true</alwaysOn>
+			  <baseline>0.11</baseline>
+			  <updateRate>$(arg f200_hz)</updateRate>
+			  <cameraName>f200</cameraName>
+			  <imageTopicName>camera/image_raw</imageTopicName>
+			  <cameraInfoTopicName>camera/camera_info</cameraInfoTopicName>
+			  <depthImageTopicName>depth/disparity</depthImageTopicName>
+			  <depthImageCameraInfoTopicName>depth/camera_info</depthImageCameraInfoTopicName>
+			  <pointCloudTopicName>depth/points</pointCloudTopicName>
+			  <frameName>f200_optical_center_link</frameName>
+			  <pointCloudCutoff>0.2</pointCloudCutoff>
+			  <pointCloudCutoffMax>1.2</pointCloudCutoffMax>
+			  <distortionK1>0.0</distortionK1>
+			  <distortionK2>0.0</distortionK2>
+			  <distortionK3>0.0</distortionK3>
+			  <distortionT1>0.0</distortionT1>
+			  <distortionT2>0.0</distortionT2>
+			  <Cx>320</Cx>
+			  <Cy>240</Cy>
+			  <focalLength>463.888592</focalLength>
+			</plugin>
+		  </sensor>
+		</gazebo>
+    </xacro:if>
   <!-- kinect 2 -->
   <xacro:if value="$(arg kinect2)">

Commit message: change elevator to torso

File: robotican_armadillo/description/models/armadillo.xacro (robot description, xacro)
@@ -6,5 +6,5 @@
 	<!--      END          -->
 	<!--    ELEV ROBOT     -->
-	<xacro:include filename="$(find robotican_armadillo)/description/models/armadillo_elevator.xacro" />
+	<xacro:include filename="$(find robotican_armadillo)/description/models/armadillo_torso.xacro" />
 	<!--      END          -->
 	<!--    ELEV ROBOT     -->
@@ -12,8 +12,8 @@
 	<!--      END          -->
 	<!--    LOAD JOINTS    -->
-	<joint name="base_elevator_joint" type="prismatic">
+	<joint name="torso_joint" type="prismatic">
 		<origin xyz="-0.1403 0 0.49381" rpy="0 0 0" />
 		<parent link="base_link" />
-		<child link="base_elevator_link" />
+		<child link="torso_link" />
 		<axis xyz="0 0 1" />
 		<dynamics damping="1000.0" friction="100000.0"/>

File: robotican_armadillo/description/models/armadillo_gazebo.xacro (robot description, xacro)
@@ -390,10 +390,10 @@
 	  </actuator>
 	</transmission>
-	<transmission name="base_elevator_joint_trans">
-	  <type>transmission_interface/SimpleTransmission</type>
-	  <joint name="base_elevator_joint">
+	<transmission name="torso_joint_trans">
+	  <type>transmission_interface/SimpleTransmission</type>
+	  <joint name="torso_joint">
 	    <hardwareInterface>PositionJointInterface</hardwareInterface>
 	  </joint>
-	  <actuator name="base_elevator_joint_motor">
+	  <actuator name="torso_joint_motor">
 	    <mechanicalReduction>1</mechanicalReduction>
 	  </actuator>
@@ -546,5 +546,5 @@
 	  </actuator>
 	</transmission>
-	<gazebo reference="base_elevator_link">
+	<gazebo reference="torso_joint_link">
 	  <turnGravityOff>true</turnGravityOff>
 	</gazebo>

File: robotican_armadillo/description/models/armadillo_torso.xacro (robot description, xacro)
@@ -1,7 +1,7 @@
 <?xml version="1.0"?>
 <robot
-  name="armadillo_elevator_urdf" description="Armadillo robot elevator">
-  <link
-    name="base_elevator_link">
+  name="armadillo_torso_urdf" description="Armadillo robot torso">
+  <link
+    name="torso_link">
     <inertial>
       <origin
@@ -24,5 +24,5 @@
       <geometry>
         <mesh
-          filename="package://robotican_armadillo/description/meshes/base_elevator_link.STL" />
+          filename="package://robotican_armadillo/description/meshes/torso_link.STL" />
       </geometry>
       <material
@@ -38,5 +38,5 @@
       <geometry>
         <mesh
-          filename="package://robotican_armadillo/description/meshes/base_elevator_link.STL" />
+          filename="package://robotican_armadillo/description/meshes/torso_link.STL" />
       </geometry>
     </collision>
@@ -89,5 +89,5 @@
       rpy="0 0 3.1416" />
     <parent
-      link="base_elevator_link" />
+      link="torso_link" />
     <child
       link="rear_cam_link" />
@@ -142,5 +142,5 @@
       rpy="0 0 0" />
     <parent
-      link="base_elevator_link" />
+      link="torso_link" />
     <child
       link="arm_link" />
@@ -195,5 +195,5 @@
       rpy="0 0 0" />
     <parent
-      link="base_elevator_link" />
+      link="torso_link" />
     <child
       link="head_link" />
