Commit message: armadillo base color change

File: robotican_armadillo/description/models/armadillo_gazebo.xacro (robot description, xacro)
@@ -634,4 +634,7 @@
   <maxVel>1.0</maxVel>
 </gazebo>
+<gazebo reference="base_link">
+    <material>Gazebo/Grey</material>
+  </gazebo>
 <gazebo reference="right_urf_link">
     <material>Gazebo/Black</material>

Commit message: komodo fixes

File: robotican_armadillo/description/models/armadillo_gazebo.xacro (robot description, xacro)
@@ -103,64 +103,4 @@
       </sensor>
     </gazebo>
-	  <!--
-	  <joint name="kinect2_head_depth_joint" type="fixed">
-	  <origin rpy="0 0 0" xyz="0.0 0.049 0.0"/>
-	  <parent link="kinect2_link"/>
-	  <child link="kinect2_head_depth_frame"/>
-	  </joint>
-	  <link name="kinect2_head_depth_frame"/>
-	  <joint name="kinect2_head_depth_optical_joint" type="fixed">
-	  <origin rpy="-1.57079632679 0.0 -1.57079632679" xyz="0 0 0"/>
-	  <parent link="kinect2_head_depth_frame"/>
-	  <child link="kinect2_head_depth_optical_frame"/>
-	  </joint>
-	  <link name="kinect2_head_depth_optical_frame"/>
-	  <joint name="kinect2_head_rgb_joint" type="fixed">
-	  <origin rpy="0 0 0" xyz="0.0 0.022 0.0"/>
-	  <parent link="kinect2_link"/>
-	  <child link="kinect2_head_rgb_frame"/>
-	  </joint>
-	  <link name="kinect2_head_rgb_frame"/>
-	  <joint name="kinect2_head_rgb_optical_joint" type="fixed">
-	  <origin rpy="-1.57079632679 0.0 -1.57079632679" xyz="0 0 0"/>
-	  <parent link="kinect2_head_rgb_frame"/>
-	  <child link="kinect2_head_rgb_optical_frame"/>
-	  </joint>
-	  <link name="kinect2_head_rgb_optical_frame"/>
-	  <gazebo reference="kinect2_head_depth_frame">
-	  <sensor name="kinect2_head" type="depth">
-	  <update_rate>20</update_rate>
-	  <camera>
-	  <horizontal_fov>1.09606677025</horizontal_fov>
-	  <image>
-	  <format>R8G8B8</format>
-	  <height>1080</height>
-	  <width>1920</width>
-	  </image>
-	  <clip>
-	  <near>0.5</near>
-	  <far>9</far>
-	  </clip>
-	  </camera>
-	  <plugin filename="libgazebo_ros_openni_kinect.so" name="kinect2_head_camera_controller">
-	  <alwaysOn>true</alwaysOn>
-	  <updateRate>20</updateRate>
-	  <imageTopicName>kinect2_head/hd/image_color</imageTopicName>
-	  <cameraInfoTopicName>kinect2_head/hd/camera_info</cameraInfoTopicName>
-	  <depthImageTopicName>kinect2_head/hd/image_depth_rect</depthImageTopicName>
-	  <depthImageCameraInfoTopicName>kinect2_head/hd/camera_info</depthImageCameraInfoTopicName>
-	  <pointCloudTopicName>kinect2_head/hd/points</pointCloudTopicName>
-	  <frameName>kinect2_head_depth_optical_frame</frameName>
-	  <distortion_k1>0.0</distortion_k1>
-	  <distortion_k2>0.0</distortion_k2>
-	  <distortion_k3>0.0</distortion_k3>
-	  <distortion_t1>0.0</distortion_t1>
-	  <distortion_t2>0.0</distortion_t2>
-	  <pointCloudCutoff>0.4</pointCloudCutoff>
-	  <pointCloudCutoffMax>50.0</pointCloudCutoffMax>
-	  </plugin>
-	  </sensor>
-	  </gazebo>
-	  -->
 	</xacro:if>
 	<!-- Sonars -->

File: robotican_komodo/description/models/komodo.xacro (robot description, xacro)
@@ -24,4 +24,60 @@
 		</collision>
 	</link>
+	  <joint name="asus_rgb_joint" type="fixed">
+      <origin xyz="0 0.022 0" rpy="0 0 0"/>
+      <parent link="asus_camera_link"/>
+      <child link="asus_rgb_frame" />
+    </joint>
+    <link name="asus_rgb_frame">
+      <inertial>
+	<mass value="0.001" />
+	<origin xyz="0 0 0" />
+	<inertia ixx="0.0001" ixy="0.0" ixz="0.0"
+	  iyy="0.0001" iyz="0.0"
+	  izz="0.0001" />
+	</inertial>
+      </link>
+      <joint name="asus_rgb_optical_joint" type="fixed">
+	<origin xyz="0 0 0" rpy="${-M_PI/2} 0 ${-M_PI/2}" />
+	<parent link="asus_rgb_frame" />
+	<child link="asus_rgb_optical_frame" />
+      </joint>
+      <link name="asus_rgb_optical_frame">
+	<inertial>
+	  <mass value="0.001" />
+	  <origin xyz="0 0 0" />
+	  <inertia ixx="0.0001" ixy="0.0" ixz="0.0"
+	    iyy="0.0001" iyz="0.0"
+	    izz="0.0001" />
+	  </inertial>
+	</link>
+	<joint name="asus_depth_joint" type="fixed">
+	  <origin xyz="0 0.049 0" rpy="0 0 0" />
+	  <parent link="asus_rgb_frame" />
+	  <child link="asus_depth_frame" />
+	</joint>
+	<link name="asus_depth_frame">
+	  <inertial>
+	    <mass value="0.001" />
+	    <origin xyz="0 0 0" />
+	    <inertia ixx="0.0001" ixy="0.0" ixz="0.0"
+	      iyy="0.0001" iyz="0.0"
+	      izz="0.0001" />
+	    </inertial>
+	  </link>
+	  <joint name="asus_depth_optical_joint" type="fixed">
+	    <origin xyz="0 0 0" rpy="${-M_PI/2} 0 ${-M_PI/2}" />
+	    <parent link="asus_depth_frame" />
+	    <child link="asus_depth_optical_frame" />
+	  </joint>
+	  <link name="asus_depth_optical_frame">
+	    <inertial>
+	      <mass value="0.001" />
+	      <origin xyz="0 0 0" />
+	      <inertia ixx="0.0001" ixy="0.0" ixz="0.0"
+		iyy="0.0001" iyz="0.0"
+		izz="0.0001" />
+	      </inertial>
+	    </link>
 	<link name="front_camera_link">
 		<inertial>

File: robotican_komodo/description/models/komodo_gazebo.xacro (robot description, xacro)
@@ -9,4 +9,46 @@
 	<xacro:arg name="gps" default="false"/>
 	<xacro:arg name="front_camera" default="false"/>
+	<xacro:arg name="asus" default="false"/>
+	  <xacro:arg name="asus_hz" default="20.0"/>
+	  <!-- asus xiton pto live -->
+  <xacro:if value="$(arg asus)">
+ <gazebo reference="asus_rgb_frame">
+      <sensor type="depth" name="asus">
+        <always_on>true</always_on>
+        <update_rate>$(arg asus_hz)</update_rate>
+      <camera>
+        <horizontal_fov>${179.0 * M_PI/180.0}</horizontal_fov>
+        <image>
+          <format>R8G8B8</format>
+          <height>640</height>
+          <width>480</width>
+        </image>
+        <clip>
+          <near>0.5</near>
+          <far>9</far>
+        </clip>
+      </camera>
+        <plugin name="asus_camera_controller" filename="libgazebo_ros_openni_kinect.so">
+          <cameraName>asus_camera</cameraName>
+          <alwaysOn>true</alwaysOn>
+          <updateRate>$(arg asus_hz)</updateRate>
+            <imageTopicName>rgb/image_raw</imageTopicName>
+            <cameraInfoTopicName>rgb/camera_info</cameraInfoTopicName>
+            <depthImageTopicName>depth/image_raw</depthImageTopicName>
+            <depthImageCameraInfoTopicName>depth/camera_info</depthImageCameraInfoTopicName>
+            <pointCloudTopicName>depth/points</pointCloudTopicName>
+          <frameName>asus_depth_optical_frame</frameName>
+          <baseline>0.1</baseline>
+    <distortion_k1>-0.02</distortion_k1>
+            <distortion_k2>0.04</distortion_k2>
+            <distortion_k3>-0.06</distortion_k3>
+            <distortion_t1>0.0</distortion_t1>
+            <distortion_t2>0.0</distortion_t2>
+       	  <pointCloudCutoff>0.4</pointCloudCutoff>
+	  <pointCloudCutoffMax>8.0</pointCloudCutoffMax>
+        </plugin>
+      </sensor>
+    </gazebo>
+	</xacro:if>
 	<!-- Sonars -->
 	<xacro:if value="$(arg urf)">
@@ -120,5 +162,5 @@
 	    <sensor type="ray" name="head_hokuyo_sensor">
 	      <pose>0 0 0 0 0 0</pose>
-	      <visualize>true</visualize>
+	      <visualize>false</visualize>
 	      <update_rate>40</update_rate>
 	      <ray>

Commit message: pick demo

File: robotican_armadillo/description/models/armadillo_gazebo.xacro (robot description, xacro)
@@ -17,6 +17,7 @@
 	  <gripper name="gripper">
 		<grasp_check>
-		  <attach_steps>5</attach_steps>
-		  <detach_steps>10</detach_steps>
+	     <attach_steps>1</attach_steps>
+	     <detach_steps>2</detach_steps>
+	     <min_contact_count>2</min_contact_count>
 		</grasp_check>
 		<gripper_link>left_finger_link</gripper_link>
@@ -25,4 +26,48 @@
 	  </gripper>
 	</gazebo>
+	<!--
+	<gazebo reference="wrist_link">
+      <kp>1000000.0</kp>
+      <kd>100.0</kd>
+      <mu1>1.0</mu1>
+      <mu2>1.0</mu2>
+      <fdir1>0 0 1</fdir1>
+      <maxVel>1.0</maxVel>
+      <minDepth>0.00</minDepth>
+      <material>Gazebo/Grey</material>
+    </gazebo>
+    <gazebo reference="wrist_joint">
+      <implicitSpringDamper>1</implicitSpringDamper>
+      <provideFeedback>1</provideFeedback>
+    </gazebo>
+    	<gazebo reference="left_finger_link">
+      <kp>1000000.0</kp>
+      <kd>100.0</kd>
+      <mu1>1.0</mu1>
+      <mu2>1.0</mu2>
+      <fdir1>0 0 1</fdir1>
+      <maxVel>1.0</maxVel>
+      <minDepth>0.00</minDepth>
+      <material>Gazebo/Grey</material>
+    </gazebo>
+    <gazebo reference="left_finger_joint">
+      <implicitSpringDamper>1</implicitSpringDamper>
+      <provideFeedback>1</provideFeedback>
+    </gazebo>
+     	<gazebo reference="right_finger_link">
+      <kp>1000000.0</kp>
+      <kd>100.0</kd>
+      <mu1>1.0</mu1>
+      <mu2>1.0</mu2>
+      <fdir1>0 0 1</fdir1>
+      <maxVel>1.0</maxVel>
+      <minDepth>0.00</minDepth>
+      <material>Gazebo/Grey</material>
+    </gazebo>
+    <gazebo reference="right_finger_joint">
+      <implicitSpringDamper>1</implicitSpringDamper>
+      <provideFeedback>1</provideFeedback>
+    </gazebo>
+	-->
   <!--  <link name="dummy_link">
   </link>
