Commit message: ekf

File: robotican_armadillo/description/models/armadillo_base.xacro (robot description, xacro)
@@ -134,5 +134,5 @@
       <geometry>
 	<!--  <mesh filename="package://robotican_armadillo/description/meshes/left_urf_link.STL" /> -->
-	<cylinder  length="0.01" radius="0.008"/>
+	<cylinder  length="0.005" radius="0.008"/>
       </geometry>
       <material

File: robotican_armadillo/description/models/armadillo_gazebo.xacro (robot description, xacro)
@@ -328,6 +328,6 @@
 	      <frameId>base_link</frameId>
 	      <topicName>IMU/data</topicName>
-	      <gaussianNoise>2.89e-08</gaussianNoise>
-	      <xyzOffsets>0 0 0</xyzOffsets>
+	      <gaussianNoise>0.1</gaussianNoise>
+	      <xyzOffsets>0 0 ${M_PI}</xyzOffsets>
 	      <rpyOffsets>0 0 0</rpyOffsets>
 	      <material>Gazebo/Red</material>

Commit message: fixes

File: robotican_armadillo/description/models/armadillo_base.xacro (robot description, xacro)
@@ -304,5 +304,5 @@
       <origin
         xyz="0 0 0"
-        rpy="1.57079632679 0 0" />
+        rpy="${M_PI/2} 0 0" />
       <geometry>
     <!--  <mesh filename="package://robotican_armadillo/description/meshes/left_wheel_link.STL" /> -->
@@ -343,5 +343,5 @@
       <origin
         xyz="0 0 0"
-         rpy="1.57079632679 0 0" />
+         rpy="${M_PI/2} 0 0" />
       <geometry>
     <!--  <mesh filename="package://robotican_armadillo/description/meshes/right_wheel_link.STL" /> -->
@@ -357,5 +357,5 @@
       <origin
         xyz="0 0 0"
-        rpy="1.57079632679 0 0" />
+        rpy="${M_PI/2} 0 0" />
       <geometry>
      <!--  <mesh filename="package://robotican_armadillo/description/meshes/right_wheel_link.STL" /> -->

File: robotican_lizi/description/models/lizi.xacro (robot description, xacro)
@@ -43,7 +43,8 @@
 			</visual>
 			<collision>
-				<origin rpy="0 0 0" xyz="0 0 0" />
-				<geometry>
-					<mesh filename="package://robotican_lizi/description/meshes/fl_wheel_link.STL" />
+				<origin rpy="${M_PI/2} 0 0" xyz="0 0 0" />
+				<geometry>
+<!-- 					<mesh filename="package://robotican_lizi/description/meshes/fl_wheel_link.STL" /> -->
+				  <cylinder  length="0.02" radius="0.065"/>
 				</geometry>
 			</collision>
@@ -65,7 +66,8 @@
 			</visual>
 			<collision>
-				<origin rpy="0 0 0" xyz="0 0 0" />
-				<geometry>
-					<mesh filename="package://robotican_lizi/description/meshes/fr_wheel_link.STL" />
+				<origin rpy="${M_PI/2} 0 0" xyz="0 0 0" />
+				<geometry>
+<!-- 					<mesh filename="package://robotican_lizi/description/meshes/fr_wheel_link.STL" /> -->
+				  <cylinder  length="0.02" radius="0.065"/>
 				</geometry>
 			</collision>
@@ -87,7 +89,8 @@
 			</visual>
 			<collision>
-				<origin rpy="0 0 0" xyz="0 0 0" />
-				<geometry>
-					<mesh filename="package://robotican_lizi/description/meshes/rl_wheel_link.STL" />
+				<origin rpy="${M_PI/2} 0 0" xyz="0 0 0" />
+				<geometry>
+<!-- 					<mesh filename="package://robotican_lizi/description/meshes/rl_wheel_link.STL" /> -->
+				  <cylinder  length="0.02" radius="0.065"/>
 				</geometry>
 			</collision>
@@ -109,7 +112,8 @@
 		</visual>
 		<collision>
-			<origin rpy="0 0 0" xyz="0 0 0" />
-			<geometry>
-				<mesh filename="package://robotican_lizi/description/meshes/rr_wheel_link.STL" />
+			<origin rpy="${M_PI/2} 0 0" xyz="0 0 0" />
+			<geometry>
+<!-- 				<mesh filename="package://robotican_lizi/description/meshes/rr_wheel_link.STL" /> -->
+			  <cylinder  length="0.02" radius="0.065"/>
 			</geometry>
 		</collision>
@@ -188,5 +192,5 @@
 		</inertial>
 		<visual>
-			<origin rpy="0 0 0" xyz="0 0 0" />
+			<origin rpy="0 0 ${M_PI}" xyz="0 0 0" />
 			<geometry>
 				<mesh filename="package://robotican_lizi/description/meshes/laser_link.STL" />
@@ -306,5 +310,5 @@
     		<child link="rl_wheel_link" />
     		<axis xyz="0 1 0" />
-    		<limit effort="0" velocity="0" />
+<!--     		<limit effort="0" velocity="0" /> -->
   	</joint>
 	<joint name="rr_wheel_joint" type="continuous">

File: robotican_lizi/description/models/lizi_gazebo.xacro (robot description, xacro)
@@ -122,8 +122,8 @@
 		<scan>
 		  <horizontal>
-		    <samples>667</samples>
-		    <resolution>1</resolution>
-		    <min_angle>-1.81</min_angle>
-		    <max_angle>1.81</max_angle>
+		    <samples>512</samples>
+		    <resolution>1</resolution>
+		    <min_angle>-1.57</min_angle>
+		    <max_angle>1.57</max_angle>
 		  </horizontal>
 		</scan>
@@ -271,3 +271,62 @@
 		</transmission>
 	</xacro:if>
+<gazebo reference="right_urf_link">
+    <material>Gazebo/Black</material>
+  </gazebo>
+  <gazebo reference="left_urf_link">
+    <material>Gazebo/Black</material>
+  </gazebo>
+    <gazebo reference="rear_urf_link">
+    <material>Gazebo/Black</material>
+  </gazebo>
+    <gazebo reference="base_link">
+    <material>Gazebo/Green</material>
+  </gazebo>
+    <gazebo reference="laser_link">
+    <material>Gazebo/Black</material>
+  </gazebo>
+  <gazebo reference="fl_wheel_link">
+    <material>Gazebo/Black</material>
+  </gazebo>
+   <gazebo reference="fr_wheel_link">
+    <material>Gazebo/Black</material>
+  </gazebo>
+    <gazebo reference="rl_wheel_link">
+    <material>Gazebo/Black</material>
+  </gazebo>
+    <gazebo reference="rr_wheel_link">
+    <material>Gazebo/Black</material>
+  </gazebo>
+  <gazebo reference="fr_wheel_link">
+  <mu1>1.0</mu1>
+  <mu2>1.0</mu2>
+  <kp>1000000.0</kp>
+  <kd>100.0</kd>
+  <minDepth>0.001</minDepth>
+  <maxVel>1.0</maxVel>
+</gazebo>
+  <gazebo reference="fl_wheel_link">
+  <mu1>1.0</mu1>
+  <mu2>1.0</mu2>
+  <kp>1000000.0</kp>
+  <kd>100.0</kd>
+  <minDepth>0.001</minDepth>
+  <maxVel>1.0</maxVel>
+</gazebo>
+  <gazebo reference="rr_wheel_link">
+  <mu1>1.0</mu1>
+  <mu2>1.0</mu2>
+  <kp>1000000.0</kp>
+  <kd>100.0</kd>
+  <minDepth>0.001</minDepth>
+  <maxVel>1.0</maxVel>
+</gazebo>
+  <gazebo reference="rl_wheel_link">
+  <mu1>1.0</mu1>
+  <mu2>1.0</mu2>
+  <kp>1000000.0</kp>
+  <kd>100.0</kd>
+  <minDepth>0.001</minDepth>
+  <maxVel>1.0</maxVel>
+</gazebo>
 </robot>

Commit message: update

File: robotican_armadillo/description/models/armadillo_base.xacro (robot description, xacro)
@@ -9,5 +9,5 @@
         rpy="0 0 0" />
       <mass
-        value="80.6548" />
+        value="180.6548" />
       <inertia
         ixx="0.61639"
@@ -32,7 +32,8 @@
       </material>
     </visual>
-      <collision name='caster_collision'>
-      <origin
-        xyz="-0.35 0 0"
+<!--
+      <collision name='caster_collision1'>
+      <origin
+        xyz="0.28 0 0"
         rpy="0 0 0" />
             <geometry>
@@ -50,12 +51,43 @@
             </surface>
           </collision>
-	<!--  <visual name='caster_visual'>
+-->
+<!--
+	  <visual name='caster_visual1'>
 	 <origin
-        xyz="-0.35 0 0"
+        xyz="0.28 0 0"
         rpy="0 0 0" />
             <geometry>
 	    <sphere radius="0.1"/>
             </geometry>
-	  </visual> -->
+	  </visual>
+-->
+      <collision name='caster_collision'>
+      <origin
+        xyz="-0.35 0 0"
+        rpy="0 0 0" />
+            <geometry>
+              <sphere radius="0.1"/>
+            </geometry>
+            <surface>
+              <friction>
+                <ode>
+                  <mu>0</mu>
+                  <mu2>0</mu2>
+                  <slip1>1.0</slip1>
+                  <slip2>1.0</slip2>
+                </ode>
+              </friction>
+            </surface>
+          </collision>
+<!--
+	  <visual name='caster_visual'>
+	 <origin
+        xyz="-0.35 0 0"
+        rpy="0 0 0" />
+            <geometry>
+	    <sphere radius="0.1"/>
+            </geometry>
+	  </visual>
+-->
   </link>
   <link

Commit message: pick done

File: robotican_armadillo/description/models/armadillo_base.xacro (robot description, xacro)
@@ -59,4 +59,10 @@
 	  </visual> -->
   </link>
+  <link name="base_footprint"/>
+ <joint name="base_link_to_base_footprint" type="fixed">
+    <parent link="base_link"/>
+    <child link="base_footprint"/>
+    <origin xyz="0.00 0.00 -0.1" rpy="0.0 0.0 0.0"/>
+  </joint>
   <link
     name="front_cam_link">

File: robotican_armadillo/description/models/armadillo_gazebo.xacro (robot description, xacro)
@@ -41,4 +41,5 @@
       <provideFeedback>1</provideFeedback>
     </gazebo>
+	-->
     	<gazebo reference="left_finger_link">
       <kp>1000000.0</kp>
@@ -69,5 +70,4 @@
       <provideFeedback>1</provideFeedback>
     </gazebo>
-	-->
   <!--  <link name="dummy_link">
   </link>
@@ -78,49 +78,4 @@
   <axis xyz="0 0 0" />
   </joint>-->
- <!--
-	<gazebo>
-   <plugin name="gazebo_grasp_fix" filename="libgazebo_grasp_fix.so">
-        <arm>
-         <gazebo>
-	  <gripper name="gripper">
-		<grasp_check>
-		  <attach_steps>5</attach_steps>
-		  <detach_steps>10</detach_steps>
-		</grasp_check>
-		<gripper_link>left_finger_link</gripper_link>
-		<gripper_link>right_finger_link</gripper_link>
-		<palm_link>wrist_link</palm_link>
-	  </gripper>
-	</gazebo>  <arm_name>arm</arm_name>
-           <palm_link> wrist_link  </palm_link>
-           <gripper_link> left_finger_link </gripper_link>
-           <gripper_link> right_finger_link </gripper_link>
-        </arm>
-       <forces_angle_tolerance>100</forces_angle_tolerance>
-       <update_rate>4</update_rate>
-       <grip_count_threshold>4</grip_count_threshold>
-       <max_grip_count>8</max_grip_count>
-       <release_tolerance>0.005</release_tolerance>
-       <disable_collisions_on_attach>false</disable_collisions_on_attach>
-       <contact_topic>__default_topic__</contact_topic>
-    </plugin>
-</gazebo>
-   <gazebo reference="right_finger_joint">
-    <implicitSpringDamper>1</implicitSpringDamper>
-      <kp>1000000.0</kp>
-  <kd>1.0</kd>
-  <mu1>1.0</mu1>
-  <mu2>1.0</mu2>
-  <minDepth>0.001</minDepth>
-  </gazebo>
-   <gazebo reference="left_finger_joint">
-    <implicitSpringDamper>1</implicitSpringDamper>
-      <kp>1000000.0</kp>
-  <kd>1.0</kd>
-  <mu1>1.0</mu1>
-  <mu2>1.0</mu2>
-  <minDepth>0.001</minDepth>
-  </gazebo>
-  -->
      <xacro:if value="$(arg f200)">
 		<gazebo reference="f200_rgb_frame">

Commit message: button update

File: robotican_armadillo/description/models/armadillo_base.xacro (robot description, xacro)
@@ -9,5 +9,5 @@
         rpy="0 0 0" />
       <mass
-        value="180.6548" />
+        value="100.6548" />
       <inertia
         ixx="0.61639"
@@ -32,8 +32,7 @@
       </material>
     </visual>
-<!--
-      <collision name='caster_collision1'>
-      <origin
-        xyz="0.28 0 0"
+      <collision name='caster_collision'>
+      <origin
+        xyz="-0.35 0 0"
         rpy="0 0 0" />
             <geometry>
@@ -51,44 +50,19 @@
             </surface>
           </collision>
--->
-<!--
-	  <visual name='caster_visual1'>
+	<!--  <visual name='caster_visual'>
 	 <origin
-        xyz="0.28 0 0"
+        xyz="-0.35 0 0"
         rpy="0 0 0" />
             <geometry>
 	    <sphere radius="0.1"/>
             </geometry>
-	  </visual>
--->
-      <collision name='caster_collision'>
-      <origin
-        xyz="-0.35 0 0"
-        rpy="0 0 0" />
-            <geometry>
-              <sphere radius="0.1"/>
-            </geometry>
-            <surface>
-              <friction>
-                <ode>
-                  <mu>0</mu>
-                  <mu2>0</mu2>
-                  <slip1>1.0</slip1>
-                  <slip2>1.0</slip2>
-                </ode>
-              </friction>
-            </surface>
-          </collision>
-<!--
-	  <visual name='caster_visual'>
-	 <origin
-        xyz="-0.35 0 0"
-        rpy="0 0 0" />
-            <geometry>
-	    <sphere radius="0.1"/>
-            </geometry>
-	  </visual>
--->
-  </link>
+	  </visual> -->
+  </link>
+  <link name="base_footprint"/>
+ <joint name="base_link_to_base_footprint" type="fixed">
+    <parent link="base_link"/>
+    <child link="base_footprint"/>
+    <origin xyz="0.00 0.00 -0.1" rpy="0.0 0.0 0.0"/>
+  </joint>
   <link
     name="front_cam_link">

File: robotican_armadillo/description/models/armadillo_gazebo.xacro (robot description, xacro)
@@ -14,4 +14,60 @@
   <xacro:arg name="kinect2_hz" default="10.0"/>
   <xacro:arg name="f200_hz" default="10.0"/>
+  <gazebo>
+	  <gripper name="gripper">
+		<grasp_check>
+	     <attach_steps>1</attach_steps>
+	     <detach_steps>2</detach_steps>
+	     <min_contact_count>2</min_contact_count>
+		</grasp_check>
+		<gripper_link>left_finger_link</gripper_link>
+		<gripper_link>right_finger_link</gripper_link>
+		<palm_link>wrist_link</palm_link>
+	  </gripper>
+	</gazebo>
+	<!--
+	<gazebo reference="wrist_link">
+      <kp>1000000.0</kp>
+      <kd>100.0</kd>
+      <mu1>1.0</mu1>
+      <mu2>1.0</mu2>
+      <fdir1>0 0 1</fdir1>
+      <maxVel>1.0</maxVel>
+      <minDepth>0.00</minDepth>
+      <material>Gazebo/Grey</material>
+    </gazebo>
+    <gazebo reference="wrist_joint">
+      <implicitSpringDamper>1</implicitSpringDamper>
+      <provideFeedback>1</provideFeedback>
+    </gazebo>
+	-->
+    	<gazebo reference="left_finger_link">
+      <kp>1000000.0</kp>
+      <kd>100.0</kd>
+      <mu1>1.0</mu1>
+      <mu2>1.0</mu2>
+      <fdir1>0 0 1</fdir1>
+      <maxVel>1.0</maxVel>
+      <minDepth>0.00</minDepth>
+      <material>Gazebo/Grey</material>
+    </gazebo>
+    <gazebo reference="left_finger_joint">
+      <implicitSpringDamper>1</implicitSpringDamper>
+      <provideFeedback>1</provideFeedback>
+    </gazebo>
+     	<gazebo reference="right_finger_link">
+      <kp>1000000.0</kp>
+      <kd>100.0</kd>
+      <mu1>1.0</mu1>
+      <mu2>1.0</mu2>
+      <fdir1>0 0 1</fdir1>
+      <maxVel>1.0</maxVel>
+      <minDepth>0.00</minDepth>
+      <material>Gazebo/Grey</material>
+    </gazebo>
+    <gazebo reference="right_finger_joint">
+      <implicitSpringDamper>1</implicitSpringDamper>
+      <provideFeedback>1</provideFeedback>
+    </gazebo>
   <!--  <link name="dummy_link">
   </link>
@@ -30,5 +86,5 @@
 			  <horizontal_fov>1.20772254</horizontal_fov>
 			  <image>
-				<format>R8G8B8</format>
+				<format>B8G8R8</format>
 				<width>640</width>
 				<height>480</height>
@@ -73,5 +129,5 @@
         <horizontal_fov>1.09606677025</horizontal_fov>
         <image>
-          <format>R8G8B8</format>
+          <format>B8G8R8</format>
           <height>1080</height>
           <width>1920</width>
@@ -86,10 +142,10 @@
           <alwaysOn>true</alwaysOn>
           <updateRate>$(arg kinect2_hz)</updateRate>
-	  <imageTopicName>hd/image_color</imageTopicName>
-	  <cameraInfoTopicName>hd/camera_info</cameraInfoTopicName>
-	  <depthImageTopicName>hd/image_depth_rect</depthImageTopicName>
-	  <depthImageCameraInfoTopicName>hd/camera_info</depthImageCameraInfoTopicName>
-	  <pointCloudTopicName>hd/points</pointCloudTopicName>
-          <frameName>kinect2_depth_optical_frame</frameName>
+	      <imageTopicName>hd/image_color</imageTopicName>
+	      <cameraInfoTopicName>hd/camera_info</cameraInfoTopicName>
+	      <depthImageTopicName>hd/image_depth_rect</depthImageTopicName>
+	      <depthImageCameraInfoTopicName>hd/camera_info</depthImageCameraInfoTopicName>
+	      <pointCloudTopicName>hd/points</pointCloudTopicName>
+		  <frameName>kinect2_depth_optical_frame</frameName>
           <baseline>0.1</baseline>
           <distortion_k1>0.0</distortion_k1>
@@ -99,5 +155,5 @@
           <distortion_t2>0.0</distortion_t2>
        	  <pointCloudCutoff>0.4</pointCloudCutoff>
-	  <pointCloudCutoffMax>8.0</pointCloudCutoffMax>
+		  <pointCloudCutoffMax>8.0</pointCloudCutoffMax>
         </plugin>
       </sensor>
