Commit message: building lizi

File: robotican_lizi/description/models/lizi_base.xacro (robot description, xacro)
@@ -1,20 +1,322 @@
 <?xml version="1.0"?>
-<robot xmlns:xacro="http://www.ros.org/wiki/xacro" name="komodo">
+<robot xmlns:xacro="http://www.ros.org/wiki/xacro" name="lizi">
 	<!-- Load all the links  -->
-	<xacro:arg name="wheels_type" default="fixed"/>
 	<xacro:arg name="have_pan_tilt" default="false"/>
 	<xacro:property name="lizi_color" value="0 0.517 0.26 1" />
-	<xacro:include filename="$(find robotican_description)/lizi/lizi_links/lizi_rover.xacro" />
+	<link name="base_link">
+			<inertial>
+				<origin rpy="0 0 0" xyz="-0.036889 0.00027038 0.069426" />
+				<mass value="4.706" />
+				<inertia ixx="0.032024" ixy="0.00038846" ixz="-0.0046108" iyy="0.065583" iyz="2.8552E-06" izz="0.076391" />
+			</inertial>
+			<visual>
+				<origin rpy="0 0 0" xyz="0 0 0" />
+				<geometry>
+					<mesh filename="package://robotican_lizi/description/meshes/base_link.STL" />
+				</geometry>
+				<material name="">
+					<color rgba="${lizi_color}" />
+				</material>
+			</visual>
+			<collision>
+				<origin rpy="0 0 0" xyz="0 0 0" />
+				<geometry>
+					<mesh filename="package://robotican_lizi/description/meshes/base_link.STL" />
+				</geometry>
+			</collision>
+	</link>
+	<link name="fl_wheel_link">
+			<inertial>
+				<origin rpy="0 0 0" xyz="2.9411E-11 -0.0075967 5.8231E-11" />
+				<mass value="0.4084" />
+				<inertia ixx="0.00059356" ixy="3.4979E-14" ixz="-4.6514E-14" iyy="0.0011268" iyz="5.6928E-14" izz="0.00059356" />
+			</inertial>
+			<visual>
+				<origin rpy="0 0 0" xyz="0 0 0" />
+				<geometry>
+					<mesh filename="package://robotican_lizi/description/meshes/fl_wheel_link.STL" />
+				</geometry>
+				<material name="">
+					<color rgba="0.2 0.2 0.2 1" />
+				</material>
+			</visual>
+			<collision>
+				<origin rpy="0 0 0" xyz="0 0 0" />
+				<geometry>
+					<mesh filename="package://robotican_lizi/description/meshes/fl_wheel_link.STL" />
+				</geometry>
+			</collision>
+	</link>
+	<link name="fr_wheel_link">
+			<inertial>
+				<origin rpy="0 0 0" xyz="-2.9052E-11 0.0035967 5.8411E-11" />
+				<mass value="0.4084" />
+				<inertia ixx="0.00059356" ixy="3.4627E-14" ixz="4.9977E-14" iyy="0.0011268" iyz="-5.7142E-14" izz="0.00059356" />
+			</inertial>
+			<visual>
+				<origin rpy="0 0 0" xyz="0 0 0" />
+				<geometry>
+					<mesh filename="package://robotican_lizi/description/meshes/fr_wheel_link.STL" />
+				</geometry>
+				<material name="">
+					<color rgba="0.2 0.2 0.2 1" />
+				</material>
+			</visual>
+			<collision>
+				<origin rpy="0 0 0" xyz="0 0 0" />
+				<geometry>
+					<mesh filename="package://robotican_lizi/description/meshes/fr_wheel_link.STL" />
+				</geometry>
+			</collision>
+	</link>
+	<link name="rl_wheel_link">
+			<inertial>
+				<origin rpy="0 0 0" xyz="2.9411E-11 -0.0035967 5.8231E-11" />
+				<mass value="0.4084" />
+				<inertia ixx="0.00059356" ixy="3.4979E-14" ixz="-4.6514E-14" iyy="0.0011268" iyz="5.6928E-14" izz="0.00059356" />
+			</inertial>
+			<visual>
+				<origin rpy="0 0 0" xyz="0 0 0" />
+				<geometry>
+					<mesh filename="package://robotican_lizi/description/meshes/rl_wheel_link.STL" />
+				</geometry>
+				<material name="">
+					<color rgba="0.2 0.2 0.2 1" />
+				</material>
+			</visual>
+			<collision>
+				<origin rpy="0 0 0" xyz="0 0 0" />
+				<geometry>
+					<mesh filename="package://robotican_lizi/description/meshes/rl_wheel_link.STL" />
+				</geometry>
+			</collision>
+	</link>
+	<link name="rr_wheel_link">
+		<inertial>
+			<origin rpy="0 0 0" xyz="-2.9411E-11 0.0035967 5.8231E-11" />
+			<mass value="0.4084" />
+			<inertia ixx="0.00059356" ixy="3.4979E-14" ixz="4.6514E-14" iyy="0.0011268" iyz="-5.6928E-14" izz="0.00059356" />
+		</inertial>
+		<visual>
+			<origin rpy="0 0 0" xyz="0 0 0" />
+			<geometry>
+				<mesh filename="package://robotican_lizi/description/meshes/rr_wheel_link.STL" />
+			</geometry>
+			<material name="">
+				<color rgba="0.2 0.2 0.2 1" />
+			</material>
+		</visual>
+		<collision>
+			<origin rpy="0 0 0" xyz="0 0 0" />
+			<geometry>
+				<mesh filename="package://robotican_lizi/description/meshes/rr_wheel_link.STL" />
+			</geometry>
+		</collision>
+  	</link>
+	<link name="right_urf_link">
+		<inertial>
+			<origin rpy="0 0 0" xyz="1.6494E-05 0.012085 -1.486E-07" />
+			<mass value="0.0020317" />
+			<inertia ixx="8.4324E-08" ixy="1.1443E-10" ixz="1.6171E-09" iyy="9.8652E-08" iyz="-1.0309E-12" izz="7.8496E-08" />
+		</inertial>
+		<visual>
+			<origin rpy="0 0 1.57" xyz="0 0 0" />
+			<geometry>
+				<mesh filename="package://robotican_lizi/description/meshes/right_urf_link.STL" />
+			</geometry>
+			<material name="">
+				<color rgba="0.19216 0.11961 0.13333 1" />
+			</material>
+		</visual>
+		<collision>
+			<origin rpy="0 0 0" xyz="0 0 0" />
+			<geometry>
+				<mesh filename="package://robotican_lizi/description/meshes/right_urf_link.STL" />
+			</geometry>
+		</collision>
+	</link>
+	<link name="rear_urf_link">
+		<inertial>
+			<origin rpy="0 0 0" xyz="0.012085 -1.486E-07 1.6494E-05" />
+			<mass value="0.0020317" />
+			<inertia ixx="9.8652E-08" ixy="-1.0309E-12" ixz="1.1443E-10" iyy="7.8496E-08" iyz="1.6171E-09" izz="8.4324E-08" />
+		</inertial>
+		<visual>
+			<origin rpy="0 0 3.14" xyz="0 0 0" />
+			<geometry>
+				<mesh filename="package://robotican_lizi/description/meshes/rear_urf_link.STL" />
+			</geometry>
+			<material name="">
+				<color rgba="0.19216 0.11961 0.13333 1" />
+			</material>
+		</visual>
+		<collision>
+			<origin rpy="0 0 0" xyz="0 0 0" />
+			<geometry>
+				<mesh filename="package://robotican_lizi/description/meshes/rear_urf_link.STL" />
+			</geometry>
+		</collision>
+	</link>
+	<link name="left_urf_link">
+		<inertial>
+			<origin rpy="0 0 0" xyz="1.6494E-05 -0.012085 1.486E-07" />
+			<mass value="0.0020317" />
+			<inertia ixx="8.4324E-08" ixy="-1.1443E-10" ixz="-1.6171E-09" iyy="9.8652E-08" iyz="-1.0309E-12" izz="7.8496E-08" />
+		</inertial>
+		<visual>
+			<origin rpy="0 0 -1.57" xyz="0 0 0" />
+			<geometry>
+				<mesh filename="package://robotican_lizi/description/meshes/left_urf_link.STL" />
+			</geometry>
+			<material name="">
+				<color rgba="0.19216 0.11961 0.13333 1" />
+			</material>
+		</visual>
+		<collision>
+			<origin rpy="0 0 0" xyz="0 0 0" />
+			<geometry>
+				<mesh filename="package://robotican_lizi/description/meshes/left_urf_link.STL" />
+			</geometry>
+		</collision>
+	</link>
+	<link name="laser_link">
+		<inertial>
+			<origin rpy="0 0 0" xyz="0.00079194 -0.00016941 -0.032844" />
+			<mass value="0.13934" />
+			<inertia ixx="7.4677E-05" ixy="-1.0667E-07" ixz="-9.0925E-07" iyy="7.7824E-05" iyz="5.076E-07" izz="5.1196E-05" />
+		</inertial>
+		<visual>
+			<origin rpy="0 0 0" xyz="0 0 0" />
+			<geometry>
+				<mesh filename="package://robotican_lizi/description/meshes/laser_link.STL" />
+			</geometry>
+			<material name="">
+				<color rgba="0.25294 0.25294 0.25294 1" />
+			</material>
+		</visual>
+		<collision>
+			<origin rpy="0 0 0" xyz="0 0 0" />
+			<geometry>
+				<mesh filename="package://robotican_lizi/description/meshes/laser_link.STL" />
+			</geometry>
+		</collision>
+	</link>
+	<link name="camera_link">
+		<inertial>
+			<origin rpy="0 0 0" xyz="-0.010925 -4.5428E-06 0.00024772" />
+			<mass value="0.033156" />
+			<inertia ixx="9.3903E-06" ixy="-1.4061E-09" ixz="5.0587E-08" iyy="5.845E-06" iyz="-2.4174E-09" izz="5.8692E-06" />
+		</inertial>
+		<visual>
+			<origin rpy="0 0 0" xyz="0 0 0" />
+			<geometry>
+				<mesh filename="package://robotican_lizi/description/meshes/camera_link.STL" />
+			</geometry>
+			<material name="">
+				<color rgba="0.2 0.2 0.2 1" />
+			</material>
+		</visual>
+		<collision>
+			<origin rpy="0 0 0" xyz="0 0 0" />
+			<geometry>
+				<mesh filename="package://robotican_lizi/description/meshes/camera_link.STL" />
+			</geometry>
+		</collision>
+	</link>
+	<link name="asus_pan_link">
+		<inertial>
+			<origin rpy="0 0 0" xyz="-0.015533 -0.010751 0.019512" />
+			<mass value="0.016162" />
+			<inertia ixx="5.2781E-06" ixy="1.178E-06" ixz="1.1286E-06" iyy="6.0052E-06" iyz="7.9421E-07" izz="4.7257E-06" />
+		</inertial>
+		<visual>
+			<origin rpy="0 0 0" xyz="0 0 0" />
+			<geometry>
+				<mesh filename="package://robotican_lizi/description/meshes/asus_pan_link.STL" />
+			</geometry>
+			<material name="">
+				<color rgba="0.2 0.2 0.2 1" />
+			</material>
+		</visual>
+		<collision>
+			<origin rpy="0 0 0" xyz="0 0 0" />
+			<geometry>
+				<mesh filename="package://robotican_lizi/description/meshes/asus_pan_link.STL" />
+			</geometry>
+		</collision>
+	</link>
 	<xacro:if value="$(arg have_pan_tilt)">
-		<xacro:include filename="$(find robotican_description)/lizi/lizi_links/Asus_Camera_link.xacro" />
-		<xacro:include filename="$(find robotican_description)/lizi/lizi_links/Asus_Pan_link.xacro" />
+		<link name="asus_camera_link">
+			<inertial>
+				<origin rpy="0 0 0" xyz="-0.00010275 -0.00025849 0.00032822" />
+				<mass value="0.14689" />
+				<inertia ixx="0.00037709" ixy="-2.2879E-08" ixz="1.0241E-05" iyy="0.00038351" iyz="1.2981E-08" izz="2.2432E-05" />
+			</inertial>
+			<visual>
+				<origin rpy="1.57 0 0" xyz="0 0 0" />
+				<geometry>
+					<mesh filename="package://robotican_lizi/description/meshes/asus_camera_link.STL" />
+				</geometry>
+				<material name="">
+					<color rgba="0.2 0.2 0.2 1" />
+				</material>
+			</visual>
+			<collision>
+				<origin rpy="0 0 0" xyz="0 0 0" />
+				<geometry>
+					<mesh filename="package://robotican_lizi/description/meshes/asus_camera_link.STL" />
+				</geometry>
+			</collision>
+		</link>
+		<link name="asus_pan_link">
+			<inertial>
+				<origin rpy="0 0 0" xyz="-0.015533 -0.010751 0.019512" />
+				<mass value="0.016162" />
+				<inertia ixx="5.2781E-06" ixy="1.178E-06" ixz="1.1286E-06" iyy="6.0052E-06" iyz="7.9421E-07" izz="4.7257E-06" />
+			</inertial>
+			<visual>
+				<origin rpy="0 0 0" xyz="0 0 0" />
+				<geometry>
+					<mesh filename="package://robotican_lizi/description/meshes/asus_pan_link.STL" />
+				</geometry>
+				<material name="">
+					<color rgba="0.2 0.2 0.2 1" />
+				</material>
+			</visual>
+			<collision>
+				<origin rpy="0 0 0" xyz="0 0 0" />
+				<geometry>
+					<mesh filename="package://robotican_lizi/description/meshes/asus_pan_link.STL" />
+				</geometry>
+			</collision>
+		</link>
 	</xacro:if>
-	<xacro:include filename="$(find robotican_description)/lizi/lizi_links/Camera_link.xacro" />
-	<xacro:include filename="$(find robotican_description)/lizi/lizi_links/Laser_link.xacro" />
-	<xacro:include filename="$(find robotican_description)/lizi/lizi_links/Left_URF_link.xacro" />
-	<xacro:include filename="$(find robotican_description)/lizi/lizi_links/Rear_URF_link.xacro" />
-	<xacro:include filename="$(find robotican_description)/lizi/lizi_links/Right_URF_link.xacro" />
 	<!--         END         -->
 	<!-- Load all the joints -->
+	<joint name="fl_wheel_Joint" type="continuous">
+    		<origin xyz="0.118 0.1338 0.026" rpy="0 0 -1.3371E-16" />
+    		<parent link="base_link" />
+    		<child link="fl_wheel_link" />
+    		<axis xyz="0 1 0" />
+  	</joint>
+	<joint name="rl_wheel_Joint" type="continuous">
+    		<origin xyz="-0.118 0.1338 0.026" rpy="0 0 -6.6853E-16" />
+    		<parent link="base_link" />
+    		<child link="rl_wheel_link" />
+    		<axis xyz="0 1 0" />
+    		<limit effort="0" velocity="0" />
+  	</joint>
+	<joint name="rr_wheel_Joint" type="continuous">
+    		<origin xyz="-0.118 -0.1338 0.026" rpy="-1.2938E-16 -1.2938E-15 -6.6853E-16" />
+    		<parent link="base_link" />
+    		<child link="rr_wheel_link" />
+    		<axis xyz="0 1 0" />
+  	</joint>
+	<joint name="fr_wheel_Joint" type="continuous">
+    		<origin xyz="0.118 -0.1338 0.026" rpy="4.4216E-16 -0.0061583 -2.6824E-16" />
+    		<parent link="base_link" />
+    		<child link="fr_wheel_link" />
+    		<axis xyz="0 1 0" />
+  	</joint>
 	<xacro:if value="$(arg have_pan_tilt)">
 		<joint name="Asus_Pan_Joint" type="fixed">
