Commit message: update

File: robotican_lizi/description/models/lizi.xacro (robot description, xacro)
@@ -1,7 +1,8 @@
 <?xml version="1.0"?>
 <robot xmlns:xacro="http://www.ros.org/wiki/xacro" name="lizi">
-	<!-- Load all the links  -->
+	<xacro:property name="M_PI" value="3.1415926535897931" />
 	<xacro:arg name="have_pan_tilt" default="false"/>
 	<xacro:property name="lizi_color" value="0 0.517 0.26 1" />
+	<!-- Load all the links  -->
 	<link name="base_link">
 			<inertial>

Commit message: update

File: robotican_lizi/description/models/lizi.xacro (robot description, xacro)
@@ -295,5 +295,5 @@
 	<!--         END         -->
 	<!-- Load all the joints -->
-	<joint name="fl_wheel_Joint" type="continuous">
+	<joint name="fl_wheel_joint" type="continuous">
     		<origin xyz="0.118 0.1338 0.026" rpy="0 0 -1.3371E-16" />
     		<parent link="base_link" />
@@ -301,5 +301,5 @@
     		<axis xyz="0 1 0" />
   	</joint>
-	<joint name="rl_wheel_Joint" type="continuous">
+	<joint name="rl_wheel_joint" type="continuous">
     		<origin xyz="-0.118 0.1338 0.026" rpy="0 0 -6.6853E-16" />
     		<parent link="base_link" />
@@ -308,5 +308,5 @@
     		<limit effort="0" velocity="0" />
   	</joint>
-	<joint name="rr_wheel_Joint" type="continuous">
+	<joint name="rr_wheel_joint" type="continuous">
     		<origin xyz="-0.118 -0.1338 0.026" rpy="-1.2938E-16 -1.2938E-15 -6.6853E-16" />
     		<parent link="base_link" />
@@ -314,5 +314,5 @@
     		<axis xyz="0 1 0" />
   	</joint>
-	<joint name="fr_wheel_Joint" type="continuous">
+	<joint name="fr_wheel_joint" type="continuous">
     		<origin xyz="0.118 -0.1338 0.026" rpy="4.4216E-16 -0.0061583 -2.6824E-16" />
     		<parent link="base_link" />
@@ -321,47 +321,47 @@
   	</joint>
 	<xacro:if value="$(arg have_pan_tilt)">
-		<joint name="Asus_Pan_Joint" type="fixed">
+		<joint name="asus_pan_joint" type="fixed">
 	    		<origin xyz="0.081249 0 0.092091" rpy="2.1253E-16 8.5011E-16 0" />
 	    		<parent link="base_link" />
-	    		<child link="Asus_Pan_link" />
+	    		<child link="asus_pan_link" />
 	    		<axis xyz="0 0 -1" />
 	    		<limit effort="0" velocity="0" />
 	  	</joint>
-		<joint name="Asus_Tilt_Joint" type="fixed">
+		<joint name="asus_tilt_joint" type="fixed">
 	    		<origin xyz="-0.0004889 -0.00041349 0.08" rpy="0 0 0" />
-	    		<parent link="Asus_Pan_link" />
-	    		<child link="Asus_Camera_link" />
+	    		<parent link="asus_pan_link" />
+	    		<child link="asus_camera_link" />
 	    		<axis xyz="0 1 0" />
 	    		<limit effort="0" velocity="0" />
 	  	</joint>
 	</xacro:if>
-	<joint name="Right_URF_Joint" type="fixed">
+	<joint name="right_urf_joint" type="fixed">
     		<origin xyz="-0.0074577 -0.1055 0.07895" rpy="0 2.6072E-16 -1.57" />
     		<parent link="base_link" />
-    		<child link="Right_URF_link" />
-    		<axis xyz="0 0 0" />
-  	</joint>
-	<joint name="Left_URF_Joint" type="fixed">
+    		<child link="right_urf_link" />
+    		<axis xyz="0 0 0" />
+  	</joint>
+	<joint name="left_urf_joint" type="fixed">
     		<origin xyz="-0.0074577 0.1055 0.07895" rpy="0 0 1.57" />
     		<parent link="base_link" />
-    		<child link="Left_URF_link" />
-    		<axis xyz="0 0 0" />
-  	</joint>
-	<joint name="Rear_URF_Joint" type="fixed">
+    		<child link="left_urf_link" />
+    		<axis xyz="0 0 0" />
+  	</joint>
+	<joint name="rear_urf_joint" type="fixed">
     		<origin xyz="-0.182 0.085 0.093934" rpy="0 0 3.14" />
     		<parent link="base_link" />
-    		<child link="Rear_URF_link" />
-    		<axis xyz="0 0 0" />
-  	</joint>
-	<joint name="Laser_Joint" type="fixed">
+    		<child link="rear_urf_link" />
+    		<axis xyz="0 0 0" />
+  	</joint>
+	<joint name="laser_joint" type="fixed">
     		<origin xyz="0.14276 -1.1564E-05 0.10781" rpy="2.1253E-16 8.5011E-16 -2.6741E-16" />
     		<parent link="base_link" />
-    		<child link="Laser_link" />
-    		<axis xyz="0 0 0" />
-  	</joint>
-	<joint name="Camera_Joint" type="fixed">
+    		<child link="laser_link" />
+    		<axis xyz="0 0 0" />
+  	</joint>
+	<joint name="camera_joint" type="fixed">
     		<origin xyz="0.178 0.05775 0.054305" rpy="1.6519E-18 -0.0061583 -2.6824E-16" />
     		<parent link="base_link" />
-    		<child link="Camera_link" />
+    		<child link="camera_link" />
     		<axis xyz="0 0 0" />
   	</joint>

File: robotican_lizi/description/models/lizi_gazebo.xacro (robot description, xacro)
@@ -1,4 +1,5 @@
 <?xml version="1.0"?>
 <robot xmlns:xacro="http://www.ros.org/wiki/xacro" name="lizi" description="lizi robot">
+	<xacro:include filename="$(find robotican_lizi)/description/models/lizi.xacro" />
 	<xacro:arg name="urf" default="false"/>
 	<xacro:arg name="imu" default="false"/>
@@ -112,3 +113,161 @@
 	  </gazebo>
 	</xacro:if>
+	<xacro:if value="$(arg lidar)">
+	  <gazebo reference="laser_link">
+	    <sensor type="ray" name="head_hokuyo_sensor">
+	      <pose>0 0 0 0 0 0</pose>
+	      <visualize>false</visualize>
+	      <update_rate>10</update_rate>
+	      <ray>
+		<scan>
+		  <horizontal>
+		    <samples>667</samples>
+		    <resolution>1</resolution>
+		    <min_angle>-1.81</min_angle>
+		    <max_angle>1.81</max_angle>
+		  </horizontal>
+		</scan>
+		<range>
+		  <min>0.02</min>
+		  <max>5.6</max>
+		  <resolution>0.01</resolution>
+		</range>
+		<noise>
+		  <type>gaussian</type>
+		  <mean>0.0</mean>
+		  <stddev>0.01</stddev>
+		</noise>
+	      </ray>
+	      <plugin name="gazebo_ros_head_hokuyo_controller" filename="libgazebo_ros_laser.so">
+		<topicName>scan</topicName>
+		<frameName>laser_link</frameName>
+	      </plugin>
+	    </sensor>
+	  </gazebo>
+	</xacro:if>
+	<!-- GPS   -->
+	<xacro:if value="$(arg gps)">
+	  <gazebo>
+	    <plugin name="GazeboRosGps" filename="libhector_gazebo_ros_gps.so">
+	      <updateRate>50.0</updateRate>
+	      <bodyName>base_link</bodyName>
+	      <frameId>base_link</frameId>
+	      <topicName>GPS/fix</topicName>
+	      <serviceName>SERVICE_GPS</serviceName>
+	      <velocityTopicName>GPS/fix_velocity</velocityTopicName>
+	      <gaussianNoise>2.89e-08 2.89e-08 2.89e-08</gaussianNoise>
+	      <velocityGaussianNoise>2.89e-08 2.89e-08 2.89e-08</velocityGaussianNoise>
+	    </plugin>
+	  </gazebo>
+	</xacro:if>
+	<!-- IMU   -->
+	<xacro:if value="$(arg imu)">
+	  <gazebo>
+	    <plugin name="GazeboRosImu" filename="libhector_gazebo_ros_imu.so">
+	      <alwaysOn>true</alwaysOn>
+	      <updateRate>50.0</updateRate>
+	      <bodyName>base_link</bodyName>
+	      <frameId>base_link</frameId>
+	      <topicName>IMU/data</topicName>
+	      <gaussianNoise>0.1</gaussianNoise>
+	      <xyzOffsets>0 0 ${M_PI}</xyzOffsets>
+	      <rpyOffsets>0 0 0</rpyOffsets>
+	      <material>Gazebo/Red</material>
+	    </plugin>
+	  </gazebo>
+	  <!-- Magnetic   -->
+	  <gazebo>
+	    <plugin name="GazeboRosMagnetic" filename="libhector_gazebo_ros_magnetic.so">
+	      <updateRate>50.0</updateRate>
+	      <bodyName>base_link</bodyName>
+	      <frameId>base_link</frameId>
+	      <topicName>IMU/magnetic</topicName>
+	      <offset>0 0 0</offset>
+	      <drift>0.0 0.0 0.0</drift>
+	      <gaussianNoise>1.3e-2 1.3e-2 1.3e-2</gaussianNoise>
+	    </plugin>
+	  </gazebo>
+	</xacro:if>
+	<!-- cameras  -->
+	<xacro:if value="$(arg front_camera)">
+	  <gazebo reference="camera_link">
+	    <sensor type="camera" name="front_camera">
+	      <update_rate>30.0</update_rate>
+	      <camera name="front_camera">
+		<horizontal_fov>1.3962634</horizontal_fov>
+		<image>
+		  <width>640</width>
+		  <height>480</height>
+		  <format>R8G8B8</format>
+		</image>
+		<clip>
+		  <near>0.02</near>
+		  <far>300</far>
+		</clip>
+		<noise>
+		  <type>gaussian</type>
+		  <mean>0.0</mean>
+		  <stddev>0.007</stddev>
+		</noise>
+	      </camera>
+	      <plugin name="front_camera_controller" filename="libgazebo_ros_camera.so">
+		<alwaysOn>true</alwaysOn>
+		<updateRate>0.0</updateRate>
+		<cameraName>front_camera</cameraName>
+		<imageTopicName>image_raw</imageTopicName>
+		<cameraInfoTopicName>camera_info</cameraInfoTopicName>
+		<frameName>camera_link</frameName>
+		<hackBaseline>0.07</hackBaseline>
+		<distortionK1>0.0</distortionK1>
+		<distortionK2>0.0</distortionK2>
+		<distortionK3>0.0</distortionK3>
+		<distortionT1>0.0</distortionT1>
+		<distortionT2>0.0</distortionT2>
+	      </plugin>
+	    </sensor>
+	  </gazebo>
+	</xacro:if>
+	<xacro:if value="$(arg controllers)">
+		<gazebo>
+		  <plugin name="gazebo_ros_control" filename="libgazebo_ros_control.so">
+			<robotSimType>gazebo_ros_control/RoboticanRobotHWSim</robotSimType>
+		  </plugin>
+		</gazebo>
+		<transmission name="fl_wheel_joint_trans">
+			<type>transmission_interface/SimpleTransmission</type>
+			<joint name="fl_wheel_joint">
+				<hardwareInterface>VelocityJointInterface</hardwareInterface>
+			</joint>
+			<actuator name="fl_wheel_joint_motor">
+				<mechanicalReduction>1</mechanicalReduction>
+			</actuator>
+		</transmission>
+		<transmission name="rl_wheel_joint_trans">
+			<type>transmission_interface/SimpleTransmission</type>
+			<joint name="rl_wheel_joint">
+				<hardwareInterface>VelocityJointInterface</hardwareInterface>
+			</joint>
+			<actuator name="rl_wheel_joint_motor">
+				<mechanicalReduction>1</mechanicalReduction>
+			</actuator>
+		</transmission>
+		<transmission name="rr_wheel_joint_trans">
+			<type>transmission_interface/SimpleTransmission</type>
+			<joint name="rr_wheel_joint">
+				<hardwareInterface>VelocityJointInterface</hardwareInterface>
+			</joint>
+			<actuator name="rr_wheel_joint_motor">
+				<mechanicalReduction>1</mechanicalReduction>
+			</actuator>
+		</transmission>
+		<transmission name="fr_wheel_joint_trans">
+			<type>transmission_interface/SimpleTransmission</type>
+			<joint name="fr_wheel_joint">
+				<hardwareInterface>VelocityJointInterface</hardwareInterface>
+			</joint>
+			<actuator name="fr_wheel_joint_motor">
+				<mechanicalReduction>1</mechanicalReduction>
+			</actuator>
+		</transmission>
+	</xacro:if>
 </robot>

Commit message: update

File: robotican_lizi/description/models/lizi.xacro (robot description, xacro)
@@ -225,27 +225,27 @@
 		</collision>
 	</link>
-	<link name="asus_pan_link">
-		<inertial>
-			<origin rpy="0 0 0" xyz="-0.015533 -0.010751 0.019512" />
-			<mass value="0.016162" />
-			<inertia ixx="5.2781E-06" ixy="1.178E-06" ixz="1.1286E-06" iyy="6.0052E-06" iyz="7.9421E-07" izz="4.7257E-06" />
-		</inertial>
-		<visual>
-			<origin rpy="0 0 0" xyz="0 0 0" />
-			<geometry>
-				<mesh filename="package://robotican_lizi/description/meshes/asus_pan_link.STL" />
-			</geometry>
-			<material name="">
-				<color rgba="0.2 0.2 0.2 1" />
-			</material>
-		</visual>
-		<collision>
-			<origin rpy="0 0 0" xyz="0 0 0" />
-			<geometry>
-				<mesh filename="package://robotican_lizi/description/meshes/asus_pan_link.STL" />
-			</geometry>
-		</collision>
-	</link>
 	<xacro:if value="$(arg have_pan_tilt)">
+		<link name="asus_pan_link">
+			<inertial>
+				<origin rpy="0 0 0" xyz="-0.015533 -0.010751 0.019512" />
+				<mass value="0.016162" />
+				<inertia ixx="5.2781E-06" ixy="1.178E-06" ixz="1.1286E-06" iyy="6.0052E-06" iyz="7.9421E-07" izz="4.7257E-06" />
+			</inertial>
+			<visual>
+				<origin rpy="0 0 0" xyz="0 0 0" />
+				<geometry>
+					<mesh filename="package://robotican_lizi/description/meshes/asus_pan_link.STL" />
+				</geometry>
+				<material name="">
+					<color rgba="0.2 0.2 0.2 1" />
+				</material>
+			</visual>
+			<collision>
+				<origin rpy="0 0 0" xyz="0 0 0" />
+				<geometry>
+					<mesh filename="package://robotican_lizi/description/meshes/asus_pan_link.STL" />
+				</geometry>
+			</collision>
+		</link>
 		<link name="asus_camera_link">
 			<inertial>

Commit message: fixes

File: robotican_lizi/description/models/lizi.xacro (robot description, xacro)
@@ -341,5 +341,5 @@
 	</xacro:if>
 	<joint name="right_urf_joint" type="fixed">
-    		<origin xyz="-0.0074577 -0.1055 0.07895" rpy="0 2.6072E-16 -1.57" />
+    		<origin xyz="-0.0074577 -0.11 0.07895" rpy="0 0 ${-M_PI/2}" />
     		<parent link="base_link" />
     		<child link="right_urf_link" />
@@ -347,5 +347,5 @@
   	</joint>
 	<joint name="left_urf_joint" type="fixed">
-    		<origin xyz="-0.0074577 0.1055 0.07895" rpy="0 0 1.57" />
+    		<origin xyz="-0.0074577 0.11 0.07895" rpy="0 0 ${M_PI/2}" />
     		<parent link="base_link" />
     		<child link="left_urf_link" />
@@ -353,5 +353,5 @@
   	</joint>
 	<joint name="rear_urf_joint" type="fixed">
-    		<origin xyz="-0.182 0.085 0.093934" rpy="0 0 3.14" />
+    		<origin xyz="-0.187 0.085 0.093934" rpy="0 0 ${M_PI}" />
     		<parent link="base_link" />
     		<child link="rear_urf_link" />
@@ -365,5 +365,5 @@
   	</joint>
 	<joint name="camera_joint" type="fixed">
-    		<origin xyz="0.178 0.05775 0.054305" rpy="1.6519E-18 -0.0061583 -2.6824E-16" />
+    		<origin xyz="0.18 0.05775 0.054305" rpy="1.6519E-18 -0.0061583 -2.6824E-16" />
     		<parent link="base_link" />
     		<child link="camera_link" />

File: robotican_lizi/description/models/lizi_gazebo.xacro (robot description, xacro)
@@ -298,4 +298,7 @@
     <material>Gazebo/Black</material>
   </gazebo>
+    <gazebo reference="camera_link">
+    <material>Gazebo/Black</material>
+  </gazebo>
   <gazebo reference="fr_wheel_link">
   <mu1>1.0</mu1>

Commit message: fixes

File: robotican_lizi/description/models/lizi.xacro (robot description, xacro)
@@ -148,5 +148,5 @@
 		</inertial>
 		<visual>
-			<origin rpy="0 0 3.14" xyz="0 0 0" />
+			<origin rpy="0 0 ${M_PI}" xyz="0 0 0" />
 			<geometry>
 				<mesh filename="package://robotican_lizi/description/meshes/rear_urf_link.STL" />
@@ -157,5 +157,5 @@
 		</visual>
 		<collision>
-			<origin rpy="0 0 0" xyz="0 0 0" />
+			<origin rpy="0 0 ${M_PI}" xyz="0 0 0" />
 			<geometry>
 				<mesh filename="package://robotican_lizi/description/meshes/rear_urf_link.STL" />

Commit message: added pan-tilt controller for lizi

File: robotican_lizi/description/models/lizi.xacro (robot description, xacro)
@@ -2,5 +2,4 @@
 <robot xmlns:xacro="http://www.ros.org/wiki/xacro" name="lizi">
 	<xacro:property name="M_PI" value="3.1415926535897931" />
-	<xacro:arg name="have_pan_tilt" default="false"/>
 	<xacro:property name="lizi_color" value="0 0.517 0.26 1" />
 	<!-- Load all the links  -->
@@ -229,6 +228,5 @@
 		</collision>
 	</link>
-	<xacro:if value="$(arg have_pan_tilt)">
-		<link name="asus_pan_link">
+		<link name="pan_link">
 			<inertial>
 				<origin rpy="0 0 0" xyz="-0.015533 -0.010751 0.019512" />
@@ -239,18 +237,18 @@
 				<origin rpy="0 0 0" xyz="0 0 0" />
 				<geometry>
-					<mesh filename="package://robotican_lizi/description/meshes/asus_pan_link.STL" />
-				</geometry>
-				<material name="">
-					<color rgba="0.2 0.2 0.2 1" />
-				</material>
-			</visual>
-			<collision>
-				<origin rpy="0 0 0" xyz="0 0 0" />
-				<geometry>
-					<mesh filename="package://robotican_lizi/description/meshes/asus_pan_link.STL" />
+					<mesh filename="package://robotican_lizi/description/meshes/pan_link.STL" />
+				</geometry>
+				<material name="">
+					<color rgba="0.2 0.2 0.2 1" />
+				</material>
+			</visual>
+			<collision>
+				<origin rpy="0 0 0" xyz="0 0 0" />
+				<geometry>
+					<mesh filename="package://robotican_lizi/description/meshes/pan_link.STL" />
 				</geometry>
 			</collision>
 		</link>
-		<link name="asus_camera_link">
+		<link name="rgbd_camera_link">
 			<inertial>
 				<origin rpy="0 0 0" xyz="-0.00010275 -0.00025849 0.00032822" />
@@ -259,42 +257,41 @@
 			</inertial>
 			<visual>
-				<origin rpy="1.57 0 0" xyz="0 0 0" />
-				<geometry>
-					<mesh filename="package://robotican_lizi/description/meshes/asus_camera_link.STL" />
-				</geometry>
-				<material name="">
-					<color rgba="0.2 0.2 0.2 1" />
-				</material>
-			</visual>
-			<collision>
-				<origin rpy="0 0 0" xyz="0 0 0" />
-				<geometry>
-					<mesh filename="package://robotican_lizi/description/meshes/asus_camera_link.STL" />
+				<origin rpy="${M_PI/2} 0 0" xyz="0 0 0" />
+				<geometry>
+					<mesh filename="package://robotican_lizi/description/meshes/rgbd_camera_link.STL" />
+				</geometry>
+				<material name="">
+					<color rgba="0.2 0.2 0.2 1" />
+				</material>
+			</visual>
+			<collision>
+				<origin rpy="0 0 0" xyz="0 0 0" />
+				<geometry>
+					<mesh filename="package://robotican_lizi/description/meshes/rgbd_camera_link.STL" />
 				</geometry>
 			</collision>
 		</link>
-		<link name="asus_pan_link">
-			<inertial>
-				<origin rpy="0 0 0" xyz="-0.015533 -0.010751 0.019512" />
-				<mass value="0.016162" />
-				<inertia ixx="5.2781E-06" ixy="1.178E-06" ixz="1.1286E-06" iyy="6.0052E-06" iyz="7.9421E-07" izz="4.7257E-06" />
-			</inertial>
-			<visual>
-				<origin rpy="0 0 0" xyz="0 0 0" />
-				<geometry>
-					<mesh filename="package://robotican_lizi/description/meshes/asus_pan_link.STL" />
-				</geometry>
-				<material name="">
-					<color rgba="0.2 0.2 0.2 1" />
-				</material>
-			</visual>
-			<collision>
-				<origin rpy="0 0 0" xyz="0 0 0" />
-				<geometry>
-					<mesh filename="package://robotican_lizi/description/meshes/asus_pan_link.STL" />
-				</geometry>
-			</collision>
-		</link>
-	</xacro:if>
+		<joint name="pan_joint" type="revolute">
+	    		<origin xyz="0.081249 0 0.092091" rpy="2.1253E-16 8.5011E-16 0" />
+	    		<parent link="base_link" />
+	    		<child link="pan_link" />
+	    		<axis xyz="0 0 1" />
+	    		    <limit
+      upper="0.610865"
+	  lower="-0.610865"
+      effort="1.11"
+      velocity="5.3" />
+	  	</joint>
+		<joint name="tilt_joint" type="revolute">
+	    		<origin xyz="-0.0004889 -0.00041349 0.08" rpy="0 0 0" />
+	    		<parent link="pan_link" />
+	    		<child link="rgbd_camera_link" />
+	    		<axis xyz="0 1 0" />
+	    		    <limit
+      upper="0.523599"
+	  lower="-0.523599"
+      effort="1.11"
+      velocity="5.3" />
+	  	</joint>
 	<!--         END         -->
 	<!-- Load all the joints -->
@@ -310,5 +307,4 @@
     		<child link="rl_wheel_link" />
     		<axis xyz="0 1 0" />
-<!--     		<limit effort="0" velocity="0" /> -->
   	</joint>
 	<joint name="rr_wheel_joint" type="continuous">
@@ -324,20 +320,4 @@
     		<axis xyz="0 1 0" />
   	</joint>
-	<xacro:if value="$(arg have_pan_tilt)">
-		<joint name="asus_pan_joint" type="fixed">
-	    		<origin xyz="0.081249 0 0.092091" rpy="2.1253E-16 8.5011E-16 0" />
-	    		<parent link="base_link" />
-	    		<child link="asus_pan_link" />
-	    		<axis xyz="0 0 -1" />
-	    		<limit effort="0" velocity="0" />
-	  	</joint>
-		<joint name="asus_tilt_joint" type="fixed">
-	    		<origin xyz="-0.0004889 -0.00041349 0.08" rpy="0 0 0" />
-	    		<parent link="asus_pan_link" />
-	    		<child link="asus_camera_link" />
-	    		<axis xyz="0 1 0" />
-	    		<limit effort="0" velocity="0" />
-	  	</joint>
-	</xacro:if>
 	<joint name="right_urf_joint" type="fixed">
     		<origin xyz="-0.0074577 -0.11 0.07895" rpy="0 0 ${-M_PI/2}" />

File: robotican_lizi/description/models/lizi_gazebo.xacro (robot description, xacro)
@@ -270,4 +270,22 @@
 			</actuator>
 		</transmission>
+		<transmission name="pan_joint_trans">
+	  <type>transmission_interface/SimpleTransmission</type>
+	  <joint name="pan_joint">
+	    <hardwareInterface>PositionJointInterface</hardwareInterface>
+	  </joint>
+	  <actuator name="pan_joint_motor">
+	    <mechanicalReduction>1</mechanicalReduction>
+	  </actuator>
+	</transmission>
+	<transmission name="tilt_joint_trans">
+	  <type>transmission_interface/SimpleTransmission</type>
+	  <joint name="tilt_joint">
+	    <hardwareInterface>PositionJointInterface</hardwareInterface>
+	  </joint>
+	  <actuator name="tilt_joint_motor">
+	    <mechanicalReduction>1</mechanicalReduction>
+	  </actuator>
+	</transmission>
 	</xacro:if>
 <gazebo reference="right_urf_link">
@@ -284,20 +302,26 @@
   </gazebo>
     <gazebo reference="laser_link">
-    <material>Gazebo/Black</material>
+    <material>Gazebo/FlatBlack</material>
   </gazebo>
   <gazebo reference="fl_wheel_link">
-    <material>Gazebo/Black</material>
+    <material>Gazebo/FlatBlack</material>
   </gazebo>
    <gazebo reference="fr_wheel_link">
-    <material>Gazebo/Black</material>
+    <material>Gazebo/FlatBlack</material>
   </gazebo>
     <gazebo reference="rl_wheel_link">
-    <material>Gazebo/Black</material>
+    <material>Gazebo/FlatBlack</material>
   </gazebo>
     <gazebo reference="rr_wheel_link">
-    <material>Gazebo/Black</material>
+    <material>Gazebo/FlatBlack</material>
   </gazebo>
     <gazebo reference="camera_link">
-    <material>Gazebo/Black</material>
+    <material>Gazebo/FlatBlack</material>
+  </gazebo>
+   <gazebo reference="rgbd_camera_link">
+    <material>Gazebo/FlatBlack</material>
+  </gazebo>
+     <gazebo reference="pan_link">
+    <material>Gazebo/Grey</material>
   </gazebo>
   <gazebo reference="fr_wheel_link">
