Commit message: update

File: robotican_komodo/description/models/komodo.xacro (robot description, xacro)
@@ -1,15 +1,5 @@
 <?xml version="1.0"?>
 <robot xmlns:xacro="http://www.ros.org/wiki/xacro" name="komodo">
-	<!-- Load all the links  -->
-<!--
-	<xacro:include filename="$(find robotican_description)/komodo/komodo_links/komodo_rover.xacro" />
-	<xacro:include filename="$(find robotican_description)/komodo/komodo_links/Front_Camera_link.xacro" />
-	<xacro:include filename="$(find robotican_description)/komodo/komodo_links/Asus_Camera_link.xacro" />
-	<xacro:include filename="$(find robotican_description)/komodo/komodo_links/Laser_link.xacro" />
-	<xacro:include filename="$(find robotican_description)/komodo/komodo_links/Left_URF_link.xacro" />
-	<xacro:include filename="$(find robotican_description)/komodo/komodo_links/Rear_URF_link.xacro" />
-	<xacro:include filename="$(find robotican_description)/komodo/komodo_links/Right_URF_link.xacro" />
-	<xacro:include filename="$(find robotican_description)/komodo/komodo_links/sensors_unit_link.xacro" />
--->
+	<xacro:property name="M_PI" value="3.1415926535897931" />
 	<link name="asus_camera_link">
 		<inertial>

Commit message: komodo fixes

File: robotican_komodo/description/models/komodo.xacro (robot description, xacro)
@@ -9,5 +9,5 @@
 		</inertial>
 		<visual>
-			<origin rpy="0 0 0" xyz="0 0 0" />
+			<origin rpy="0 0 0" xyz="0.005 0 0" />
 			<geometry>
 				<mesh filename="package://robotican_komodo/description/meshes/asus_camera_link.STL" />
@@ -31,5 +31,5 @@
 		</inertial>
 		<visual>
-			<origin rpy="-1.57079632649567 1.57079632649567 -1.57079632649567" xyz="0 0 0" />
+			<origin rpy="-1.57079632649567 1.57079632649567 -1.57079632649567" xyz="0.005 0 0" />
 			<geometry>
 				<mesh filename="package://robotican_komodo/description/meshes/front_camera_link.STL" />
@@ -55,5 +55,5 @@
 			<origin rpy="0 0 0" xyz="0 0 0" />
 			<geometry>
-				<mesh filename="package://robotican_komodo/description/meshes/col_base_link.STL" />
+				<mesh filename="package://robotican_komodo/description/meshes/base_link.STL" />
 			</geometry>
 			<material name="">
@@ -64,5 +64,5 @@
 			<origin rpy="0 0 0" xyz="-0.065 0 0" />
 			<geometry>
-				<mesh filename="package://robotican_komodo/description/meshes/col_base_link.STL" />
+				<mesh filename="package://robotican_komodo/description/meshes/base_link.STL" />
 			</geometry>
 		</collision>
@@ -84,7 +84,7 @@
 		</visual>
 		<collision>
-			<origin rpy="0 1.5 0" xyz="0 0 0" />
-			<geometry>
-				<cylinder length="0.05" radius="0.1" />
+			<origin rpy="0 ${M_PI/2} 0" xyz="0 0 0" />
+			<geometry>
+				<cylinder length="0.03" radius="0.1311" />
 			</geometry>
 		</collision>
@@ -106,7 +106,7 @@
 		</visual>
 		<collision>
-			<origin rpy="0 1.5 0" xyz="0 0 0" />
-			<geometry>
-				<cylinder length="0.05" radius="0.1" />
+			<origin rpy="0 ${M_PI/2} 0" xyz="0 0 0" />
+			<geometry>
+				<cylinder length="0.03" radius="0.1311" />
 			</geometry>
 		</collision>
@@ -127,8 +127,8 @@
 			</material>
 		</visual>
-   	 	<collision>
-			<origin rpy="0 1.5 0" xyz="0 0 0" />
-			<geometry>
-				<cylinder length="0.05" radius="0.1" />
+		<collision>
+			<origin rpy="0 ${M_PI/2} 0" xyz="0 0 0" />
+			<geometry>
+				<cylinder length="0.03" radius="0.1311" />
 			</geometry>
 		</collision>
@@ -150,7 +150,7 @@
 		</visual>
 		<collision>
-			<origin rpy="0 1.5 0" xyz="0 0 0" />
-			<geometry>
-				<cylinder length="0.05" radius="0.1" />
+			<origin rpy="0 ${M_PI/2} 0" xyz="0 0 0" />
+			<geometry>
+				<cylinder length="0.03" radius="0.1311" />
 			</geometry>
 		</collision>
@@ -163,5 +163,5 @@
 		</inertial>
 		<visual>
-			<origin rpy="0 0 0" xyz="0 0 0" />
+			<origin rpy="0 0 ${M_PI}" xyz="0.003 0 0" />
 			<geometry>
 				<mesh filename="package://robotican_komodo/description/meshes/laser_link.STL" />

File: robotican_komodo/description/models/komodo_gazebo.xacro (robot description, xacro)
@@ -284,14 +284,19 @@
 		<material>Gazebo/Black</material>
 	</gazebo>
-<!--
 	<gazebo reference="base_link">
-		<material>Gazebo/White</material>
-	</gazebo>
--->
-<!--
+		<material>Gazebo/Grey</material>
+	</gazebo>
+	<gazebo reference="sensors_unit_link">
+		<material>Gazebo/Grey</material>
+	</gazebo>
 	<gazebo reference="laser_link">
-		<material>Gazebo/FlatBlack</material>
-	</gazebo>
--->
+		<material>Gazebo/Black</material>
+	</gazebo>
+	<gazebo reference="asus_camera_link">
+		<material>Gazebo/Black</material>
+	</gazebo>
+	<gazebo reference="front_camera_link">
+		<material>Gazebo/Black</material>
+	</gazebo>
 	<gazebo reference="fl_wheel_link">
 		<material>Gazebo/FlatBlack</material>

Commit message: asus fixes

File: robotican_komodo/description/models/komodo.xacro (robot description, xacro)
@@ -9,5 +9,5 @@
 		</inertial>
 		<visual>
-			<origin rpy="0 0 0" xyz="0.005 0 0" />
+			<origin rpy="0 0 0" xyz="0.00 0 0" />
 			<geometry>
 				<mesh filename="package://robotican_komodo/description/meshes/asus_camera_link.STL" />
@@ -27,7 +27,7 @@
       <origin xyz="0 0.022 0" rpy="0 0 0"/>
       <parent link="asus_camera_link"/>
-      <child link="asus_rgb_frame" />
+      <child link="asus_camera_rgb_frame" />
     </joint>
-    <link name="asus_rgb_frame">
+    <link name="asus_camera_rgb_frame">
       <inertial>
 	<mass value="0.001" />
@@ -38,10 +38,10 @@
 	</inertial>
       </link>
-      <joint name="asus_rgb_optical_joint" type="fixed">
+      <joint name="asus_camera_rgb_optical_joint" type="fixed">
 	<origin xyz="0 0 0" rpy="${-M_PI/2} 0 ${-M_PI/2}" />
-	<parent link="asus_rgb_frame" />
-	<child link="asus_rgb_optical_frame" />
+	<parent link="asus_camera_rgb_frame" />
+	<child link="asus_camera_rgb_optical_frame" />
       </joint>
-      <link name="asus_rgb_optical_frame">
+      <link name="asus_camera_rgb_optical_frame">
 	<inertial>
 	  <mass value="0.001" />
@@ -52,10 +52,10 @@
 	  </inertial>
 	</link>
-	<joint name="asus_depth_joint" type="fixed">
+	<joint name="asus_camera_depth_joint" type="fixed">
 	  <origin xyz="0 0.049 0" rpy="0 0 0" />
-	  <parent link="asus_rgb_frame" />
-	  <child link="asus_depth_frame" />
+	  <parent link="asus_camera_link" />
+	  <child link="asus_camera_depth_frame" />
 	</joint>
-	<link name="asus_depth_frame">
+	<link name="asus_camera_depth_frame">
 	  <inertial>
 	    <mass value="0.001" />
@@ -66,10 +66,10 @@
 	    </inertial>
 	  </link>
-	  <joint name="asus_depth_optical_joint" type="fixed">
+	  <joint name="asus_camera_depth_optical_joint" type="fixed">
 	    <origin xyz="0 0 0" rpy="${-M_PI/2} 0 ${-M_PI/2}" />
-	    <parent link="asus_depth_frame" />
-	    <child link="asus_depth_optical_frame" />
+	    <parent link="asus_camera_depth_frame" />
+	    <child link="asus_camera_depth_optical_frame" />
 	  </joint>
-	  <link name="asus_depth_optical_frame">
+	  <link name="asus_camera_depth_optical_frame">
 	    <inertial>
 	      <mass value="0.001" />

File: robotican_komodo/description/models/komodo_gazebo.xacro (robot description, xacro)
@@ -10,13 +10,13 @@
 	<xacro:arg name="front_camera" default="false"/>
 	<xacro:arg name="asus" default="false"/>
-	  <xacro:arg name="asus_hz" default="20.0"/>
+	  <xacro:arg name="asus_hz" default="10.0"/>
 	  <!-- asus xiton pto live -->
   <xacro:if value="$(arg asus)">
- <gazebo reference="asus_rgb_frame">
-      <sensor type="depth" name="asus">
+ <gazebo reference="asus_camera_rgb_frame">
+      <sensor type="depth" name="asus_camera">
         <always_on>true</always_on>
         <update_rate>$(arg asus_hz)</update_rate>
       <camera>
-        <horizontal_fov>${179.0 * M_PI/180.0}</horizontal_fov>
+        <horizontal_fov>${57.0*M_PI/180.0}</horizontal_fov>
         <image>
           <format>R8G8B8</format>
@@ -25,6 +25,6 @@
         </image>
         <clip>
-          <near>0.5</near>
-          <far>9</far>
+          <near>0.01</near>
+          <far>5.0</far>
         </clip>
       </camera>
@@ -38,6 +38,5 @@
             <depthImageCameraInfoTopicName>depth/camera_info</depthImageCameraInfoTopicName>
             <pointCloudTopicName>depth/points</pointCloudTopicName>
-          <frameName>asus_depth_optical_frame</frameName>
-          <baseline>0.1</baseline>
+          <frameName>asus_camera_depth_optical_frame</frameName>
     <distortion_k1>-0.02</distortion_k1>
             <distortion_k2>0.04</distortion_k2>
@@ -45,6 +44,6 @@
             <distortion_t1>0.0</distortion_t1>
             <distortion_t2>0.0</distortion_t2>
-       	  <pointCloudCutoff>0.4</pointCloudCutoff>
-	  <pointCloudCutoffMax>8.0</pointCloudCutoffMax>
+       	  <pointCloudCutoff>0.01</pointCloudCutoff>
+	  <pointCloudCutoffMax>5.0</pointCloudCutoffMax>
         </plugin>
       </sensor>

File: robotican_lizi/description/models/lizi.xacro (robot description, xacro)
@@ -252,26 +252,82 @@
 			</collision>
 		</link>
-		<link name="rgbd_camera_link">
-			<inertial>
-				<origin rpy="0 0 0" xyz="-0.00010275 -0.00025849 0.00032822" />
+		<link name="asus_camera_link">
+			<inertial>
+				<origin rpy="0 0 0" xyz="0 0 0" />
 				<mass value="0.14689" />
 				<inertia ixx="0.00037709" ixy="-2.2879E-08" ixz="1.0241E-05" iyy="0.00038351" iyz="1.2981E-08" izz="2.2432E-05" />
 			</inertial>
 			<visual>
+				<origin rpy="${M_PI/2} 0 0" xyz="-0.007 0 0" />
+				<geometry>
+					<mesh filename="package://robotican_lizi/description/meshes/asus_camera_link.STL" />
+				</geometry>
+				<material name="">
+					<color rgba="0.2 0.2 0.2 1" />
+				</material>
+			</visual>
+			<collision>
 				<origin rpy="${M_PI/2} 0 0" xyz="0 0 0" />
 				<geometry>
-					<mesh filename="package://robotican_lizi/description/meshes/rgbd_camera_link.STL" />
-				</geometry>
-				<material name="">
-					<color rgba="0.2 0.2 0.2 1" />
-				</material>
-			</visual>
-			<collision>
-				<origin rpy="0 0 0" xyz="0 0 0" />
-				<geometry>
-					<mesh filename="package://robotican_lizi/description/meshes/rgbd_camera_link.STL" />
+					<mesh filename="package://robotican_lizi/description/meshes/asus_camera_link.STL" />
 				</geometry>
 			</collision>
 		</link>
+		  <joint name="asus_rgb_joint" type="fixed">
+      <origin xyz="0 0.022 0" rpy="0 0 0"/>
+      <parent link="asus_camera_link"/>
+      <child link="asus_camera_rgb_frame" />
+    </joint>
+    <link name="asus_camera_rgb_frame">
+      <inertial>
+	<mass value="0.001" />
+	<origin xyz="0 0 0" />
+	<inertia ixx="0.0001" ixy="0.0" ixz="0.0"
+	  iyy="0.0001" iyz="0.0"
+	  izz="0.0001" />
+	</inertial>
+      </link>
+      <joint name="asus_camera_rgb_optical_joint" type="fixed">
+	<origin xyz="0 0 0" rpy="${-M_PI/2} 0 ${-M_PI/2}" />
+	<parent link="asus_camera_rgb_frame" />
+	<child link="asus_camera_rgb_optical_frame" />
+      </joint>
+      <link name="asus_camera_rgb_optical_frame">
+	<inertial>
+	  <mass value="0.001" />
+	  <origin xyz="0 0 0" />
+	  <inertia ixx="0.0001" ixy="0.0" ixz="0.0"
+	    iyy="0.0001" iyz="0.0"
+	    izz="0.0001" />
+	  </inertial>
+	</link>
+	<joint name="asus_camera_depth_joint" type="fixed">
+	  <origin xyz="0 0.049 0" rpy="0 0 0" />
+	  <parent link="asus_camera_link" />
+	  <child link="asus_camera_depth_frame" />
+	</joint>
+	<link name="asus_camera_depth_frame">
+	  <inertial>
+	    <mass value="0.001" />
+	    <origin xyz="0 0 0" />
+	    <inertia ixx="0.0001" ixy="0.0" ixz="0.0"
+	      iyy="0.0001" iyz="0.0"
+	      izz="0.0001" />
+	    </inertial>
+	  </link>
+	  <joint name="asus_camera_depth_optical_joint" type="fixed">
+	    <origin xyz="0 0 0" rpy="${-M_PI/2} 0 ${-M_PI/2}" />
+	    <parent link="asus_camera_depth_frame" />
+	    <child link="asus_camera_depth_optical_frame" />
+	  </joint>
+	  <link name="asus_camera_depth_optical_frame">
+	    <inertial>
+	      <mass value="0.001" />
+	      <origin xyz="0 0 0" />
+	      <inertia ixx="0.0001" ixy="0.0" ixz="0.0"
+		iyy="0.0001" iyz="0.0"
+		izz="0.0001" />
+	      </inertial>
+	    </link>
 	</xacro:if>
 	<!--         END         -->
@@ -312,5 +368,5 @@
 				<origin xyz="-0.0004889 -0.00041349 0.08" rpy="0 0 0" />
 				<parent link="pan_link" />
-				<child link="rgbd_camera_link" />
+				<child link="asus_camera_link" />
 				<axis xyz="0 1 0" />
 				<limit upper="0.523599" lower="-0.523599" effort="1.11" velocity="5.3" />

File: robotican_lizi/description/models/lizi_gazebo.xacro (robot description, xacro)
@@ -8,4 +8,44 @@
 	<xacro:arg name="lidar" default="false"/>
 	<xacro:property name="URF_FOV" value="${10.0*M_PI/180}" />
+	  <xacro:arg name="asus_hz" default="10.0"/>
+		<xacro:if value="$(arg pan_tilt)">
+	  	  <!-- asus xiton pto live -->
+ <gazebo reference="asus_camera_rgb_frame">
+      <sensor type="depth" name="asus_camera">
+        <always_on>true</always_on>
+        <update_rate>$(arg asus_hz)</update_rate>
+      <camera>
+        <horizontal_fov>${57.0*M_PI/180.0}</horizontal_fov>
+        <image>
+          <format>R8G8B8</format>
+          <height>640</height>
+          <width>480</width>
+        </image>
+        <clip>
+          <near>0.01</near>
+          <far>5.0</far>
+        </clip>
+      </camera>
+        <plugin name="asus_camera_controller" filename="libgazebo_ros_openni_kinect.so">
+          <cameraName>asus_camera</cameraName>
+          <alwaysOn>true</alwaysOn>
+          <updateRate>$(arg asus_hz)</updateRate>
+            <imageTopicName>rgb/image_raw</imageTopicName>
+            <cameraInfoTopicName>rgb/camera_info</cameraInfoTopicName>
+            <depthImageTopicName>depth/image_raw</depthImageTopicName>
+            <depthImageCameraInfoTopicName>depth/camera_info</depthImageCameraInfoTopicName>
+            <pointCloudTopicName>depth/points</pointCloudTopicName>
+          <frameName>asus_camera_depth_optical_frame</frameName>
+    <distortion_k1>-0.02</distortion_k1>
+            <distortion_k2>0.04</distortion_k2>
+            <distortion_k3>-0.06</distortion_k3>
+            <distortion_t1>0.0</distortion_t1>
+            <distortion_t2>0.0</distortion_t2>
+       	  <pointCloudCutoff>0.01</pointCloudCutoff>
+	  <pointCloudCutoffMax>5.0</pointCloudCutoffMax>
+        </plugin>
+      </sensor>
+    </gazebo>
+    </xacro:if>
 	<xacro:if value="$(arg urf)">
 	  <gazebo reference="left_urf_link">
@@ -322,5 +362,5 @@
    </gazebo>
    <xacro:if value="$(arg pan_tilt)">
-	   <gazebo reference="rgbd_camera_link">
+	   <gazebo reference="asus_camera_link">
 		<material>Gazebo/FlatBlack</material>
 	   </gazebo>
